File: MicroPilot/MicroPilot.sch (KiCad schematic (older format))
At the start: 1 part

Commit message: MicroPilot schematic done
Parts:
- removed J?: Header, symbol Connector:Conn_01x10_Female
- added J?: Header, symbol Connector:Conn_01x08_Female
Connections:
- net +3V3: now also J?.1 (Pin_1)
- net +BATT: now also J?.3 (Pin_3)
- net GND: now also J?.2 (Pin_2), J?.4 (Pin_4)
- net UART_SBC_RX: now also J?.5 (Pin_5)
- net UART_SBC_TX: now also J?.6 (Pin_6)
Changed lines of the file:
@@
 EESchema Schematic File Version 4
+LIBS:MicroPilot-cache
 EELAYER 26 0
 EELAYER END
 $Descr A4 11693 8268
 encoding utf-8
-Sheet 1 3
+Sheet 1 2
 Title ""
 Date ""
@@
 L power:GND #PWR?
 U 1 1 5C6ED8CD
-P 2100 1700
-F 0 "#PWR?" H 2100 1450 50  0001 C CNN
-F 1 "GND" V 2105 1572 50  0000 R CNN
-F 2 "" H 2100 1700 50  0001 C CNN
-F 3 "" H 2100 1700 50  0001 C CNN
-	1    2100 1700
+P 5800 4200
+F 0 "#PWR?" H 5800 3950 50  0001 C CNN
+F 1 "GND" V 5805 4072 50  0000 R CNN
+F 2 "" H 5800 4200 50  0001 C CNN
+F 3 "" H 5800 4200 50  0001 C CNN
+	1    5800 4200
 	0    1    1    0
 $EndComp
-Text Label 2100 1800 2    50   ~ 0
+Text Label 5800 4300 2    50   ~ 0
 UART_SBC_RX
-Text Label 2100 1900 2    50   ~ 0
+Text Label 5800 4400 2    50   ~ 0
 UART_SBC_TX
-NoConn ~ 2100 2000
-NoConn ~ 2100 2100
-Text Label 2100 2200 2    50   ~ 0
-PWM_SBC_0
-Text Label 2100 2300 2    50   ~ 0
-PWM_SBC_1
-$Comp
-L Connector:Conn_01x10_Female J?
-U 1 1 5C6EDBA3
-P 2300 1800
-F 0 "J?" H 2327 1776 50  0000 L CNN
-F 1 "Header" H 2327 1685 50  0000 L CNN
-F 2 "" H 2300 1800 50  0001 C CNN
-F 3 "~" H 2300 1800 50  0001 C CNN
-	1    2300 1800
-	1    0    0    -1
-$EndComp
+NoConn ~ 5800 4500
 $Comp
 L power:+BATT #PWR?
 U 1 1 5C6EDCD1
-P 2100 1600
-F 0 "#PWR?" H 2100 1450 50  0001 C CNN
-F 1 "+BATT" V 2115 1727 50  0000 L CNN
-F 2 "" H 2100 1600 50  0001 C CNN
-F 3 "" H 2100 1600 50  0001 C CNN
-	1    2100 1600
+P 5800 4100
+F 0 "#PWR?" H 5800 3950 50  0001 C CNN
+F 1 "+BATT" V 5815 4227 50  0000 L CNN
+F 2 "" H 5800 4100 50  0001 C CNN
+F 3 "" H 5800 4100 50  0001 C CNN
+	1    5800 4100
 	0    -1   -1   0
 $EndComp
@@
 L power:GND #PWR?
 U 1 1 5C6EDD25
-P 2100 1500
-F 0 "#PWR?" H 2100 1250 50  0001 C CNN
-F 1 "GND" V 2105 1372 50  0000 R CNN
-F 2 "" H 2100 1500 50  0001 C CNN
-F 3 "" H 2100 1500 50  0001 C CNN
-	1    2100 1500
+P 5800 4000
+F 0 "#PWR?" H 5800 3750 50  0001 C CNN
+F 1 "GND" V 5805 3872 50  0000 R CNN
+F 2 "" H 5800 4000 50  0001 C CNN
+F 3 "" H 5800 4000 50  0001 C CNN
+	1    5800 4000
 	0    1    1    0
 $EndComp
@@
 L power:+3.3V #PWR?
 U 1 1 5C6EDD8A
-P 2100 1400
-F 0 "#PWR?" H 2100 1250 50  0001 C CNN
-F 1 "+3.3V" V 2115 1528 50  0000 L CNN
-F 2 "" H 2100 1400 50  0001 C CNN
-F 3 "" H 2100 1400 50  0001 C CNN
-	1    2100 1400
+P 5800 3900
+F 0 "#PWR?" H 5800 3750 50  0001 C CNN
+F 1 "+3.3V" V 5815 4028 50  0000 L CNN
+F 2 "" H 5800 3900 50  0001 C CNN
+F 3 "" H 5800 3900 50  0001 C CNN
+	1    5800 3900
 	0    -1   -1   0
 $EndComp
-$Sheet
-S 7900 800  1350 1900
-U 5C6EDE9F
-F0 "Power" 50
-F1 "Power.sch" 50
-$EndSheet
 $Sheet
 S 7900 3850 1350 1600
@@
 F0 "FlightControler" 50
 F1 "FC.sch" 50
+F2 "MAIN_UART_RX" I L 7900 4150 50
+F3 "MAIN_UART_TX" O L 7900 4350 50
 $EndSheet
+$Comp
+L Connector:Conn_01x08_Female J?
+U 1 1 5C718E23
+P 6000 4200
+F 0 "J?" H 6027 4176 50  0000 L CNN
+F 1 "Header" H 6027 4085 50  0000 L CNN
+F 2 "" H 6000 4200 50  0001 C CNN
+F 3 "~" H 6000 4200 50  0001 C CNN
+	1    6000 4200
+	1    0    0    -1
+$EndComp
+NoConn ~ 5800 4600
+Text Label 7900 4350 2    50   ~ 0
+UART_SBC_RX
+Text Label 7900 4150 2    50   ~ 0
+UART_SBC_TX
 $EndSCHEMATC
