File: OB/io.sch (KiCad schematic (older format))
At the start: 24 parts, among them U1 V3S, U4 MX25L12835E, Y1 X1E0000210832, Y2 CC5V-T1A 32.768KHZ +-20PPM 12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

Commit message: Progress on wifi
Parts:
- removed J?: Micro_SD_Card_Det, symbol Connector:Micro_SD_Card_Det
- removed J?: Header, symbol Connector:Conn_01x06_Female
- removed U?: AR9271, symbol ob:AR9271
- added J?: CAM, symbol Connector:Conn_01x24_Female
- added J?: Header, symbol Connector:Conn_01x08_Female
- added R? (x2): 5.1K, symbol Device:R
- added TP?: USB_ID, symbol Connector:TestPoint
- added TP?: USB_DN, symbol Connector:TestPoint
- added TP?: USB_DP, symbol Connector:TestPoint
Connections:
- net labels added: +1V8, +2V8, +BATT, CSI_HSYNC, CSI_I2C_SCL, CSI_I2C_SDA, CSI_MCLK, CSI_PCLK, CSI_PWDN, CSI_VSYNC, CSI_Y0, CSI_Y1, CSI_Y2, CSI_Y3, CSI_Y4, CSI_Y5, CSI_Y6, CSI_Y7, CSI_Y8, CSI_Y9, DVDD, PWM0, PWM1, ~CSI_RST
- net labels removed: USB_DRVVBUS, VBAT
- wire segments 41 -> 44
- no-connect marks 57 -> 39
Other:
- moved on the sheet: C33, C36, C37, C38, C40, C41, R29, R30, R?, TP4, Y1, Y2

Commit message: wifi antenna done
Parts:
- removed TP?: USB_ID, symbol Connector:TestPoint
- removed TP?: USB_DN, symbol Connector:TestPoint
- removed TP?: USB_DP, symbol Connector:TestPoint
- added J?: PROG, symbol Connector:Conn_01x05_Female
Connections:
- net +BATT: now also J?.4 (Pin_4)
- net GND: now also J?.5 (Pin_5)
- net USB_D_N: now also J?.2 (Pin_2)
- net USB_D_P: now also J?.3 (Pin_3)
- net USB_ID: now also J?.1 (Pin_1)
Changed lines of the file:
@@
 Text Label 3500 4350 0    50   ~ 0
 PWM1
-$Comp
-L Connector:TestPoint TP?
-U 1 1 5C7A3797
-P 5750 6250
-F 0 "TP?" V 5704 6437 50  0000 L CNN
-F 1 "USB_ID" V 5795 6437 50  0000 L CNN
-F 2 "" H 5950 6250 50  0001 C CNN
-F 3 "~" H 5950 6250 50  0001 C CNN
-	1    5750 6250
-	0    1    1    0
-$EndComp
-$Comp
-L Connector:TestPoint TP?
-U 1 1 5C7A38A7
-P 5750 6450
-F 0 "TP?" V 5704 6637 50  0000 L CNN
-F 1 "USB_DN" V 5795 6637 50  0000 L CNN
-F 2 "" H 5950 6450 50  0001 C CNN
-F 3 "~" H 5950 6450 50  0001 C CNN
-	1    5750 6450
-	0    1    1    0
-$EndComp
-$Comp
-L Connector:TestPoint TP?
-U 1 1 5C7A422A
-P 5750 6650
-F 0 "TP?" V 5704 6837 50  0000 L CNN
-F 1 "USB_DP" V 5795 6837 50  0000 L CNN
-F 2 "" H 5950 6650 50  0001 C CNN
-F 3 "~" H 5950 6650 50  0001 C CNN
-	1    5750 6650
-	0    1    1    0
-$EndComp
+Text HLabel 5750 6350 0    50   BiDi ~ 0
+USB_D_N
 Text HLabel 5750 6450 0    50   BiDi ~ 0
-USB_D_N
-Text HLabel 5750 6650 0    50   BiDi ~ 0
 USB_D_P
 Text HLabel 8600 5300 0    50   BiDi ~ 0
@@
 Text HLabel 8600 5500 0    50   BiDi ~ 0
 USB_D_P
+$Comp
+L Connector:Conn_01x05_Female J?
+U 1 1 5C6DACA7
+P 5950 6450
+F 0 "J?" H 5977 6476 50  0000 L CNN
+F 1 "PROG" H 5977 6385 50  0000 L CNN
+F 2 "" H 5950 6450 50  0001 C CNN
+F 3 "~" H 5950 6450 50  0001 C CNN
+	1    5950 6450
+	1    0    0    -1
+$EndComp
+$Comp
+L power:GND #PWR?
+U 1 1 5C6DD5A1
+P 5750 6650
+F 0 "#PWR?" H 5750 6400 50  0001 C CNN
+F 1 "GND" V 5755 6522 50  0000 R CNN
+F 2 "" H 5750 6650 50  0001 C CNN
+F 3 "" H 5750 6650 50  0001 C CNN
+	1    5750 6650
+	0    1    1    0
+$EndComp
+$Comp
+L power:+BATT #PWR?
+U 1 1 5C6DD5A7
+P 5750 6550
+F 0 "#PWR?" H 5750 6400 50  0001 C CNN
+F 1 "+BATT" V 5765 6677 50  0000 L CNN
+F 2 "" H 5750 6550 50  0001 C CNN
+F 3 "" H 5750 6550 50  0001 C CNN
+	1    5750 6550
+	0    -1   -1   0
+$EndComp
 $EndSCHEMATC

Commit message: SmartBridgeMicro Schematic done
Connections:
- net +3V3: now also J?.1 (Pin_1)
- net +BATT: now also J?.3 (Pin_3); no longer J?.1 (Pin_1)
- net GND: now also J?.4 (Pin_4)
- net I2C0_CLK: now also J?.7 (Pin_7); no longer J?.5 (Pin_5)
- net I2C0_SDA: now also J?.8 (Pin_8); no longer J?.6 (Pin_6)
- net UART0_RX: now also J?.5 (Pin_5); no longer J?.3 (Pin_3)
- net UART0_TX: now also J?.6 (Pin_6); no longer J?.4 (Pin_4)
- net PWM0: no longer names the net of U1.43 (PB4/PWM0)
- net PWM0: no longer J?.7 (Pin_7)
- net PWM1: no longer names the net of U1.44 (PB5/PWM1)
- net PWM1: no longer J?.8 (Pin_8)
- no-connect marks 39 -> 41
Changed lines of the file:
@@
 Text Label 3550 5100 0    50   ~ 0
 UART0_TX
-Text Label 5800 2850 2    50   ~ 0
+Text Label 5800 3050 2    50   ~ 0
 UART0_RX
-Text Label 5800 2950 2    50   ~ 0
+Text Label 5800 3150 2    50   ~ 0
 UART0_TX
 $Comp
@@
 Text Label 5600 2300 2    50   ~ 0
 I2C0_SDA
-Text Label 5800 3050 2    50   ~ 0
+Text Label 5800 3250 2    50   ~ 0
 I2C0_CLK
-Text Label 5800 3150 2    50   ~ 0
+Text Label 5800 3350 2    50   ~ 0
 I2C0_SDA
 Text Label 3500 4550 0    50   ~ 0
@@
 L power:+BATT #PWR?
 U 1 1 5C78E0EE
-P 5800 2650
-F 0 "#PWR?" H 5800 2500 50  0001 C CNN
-F 1 "+BATT" V 5815 2777 50  0000 L CNN
-F 2 "" H 5800 2650 50  0001 C CNN
-F 3 "" H 5800 2650 50  0001 C CNN
-	1    5800 2650
+P 5800 2850
+F 0 "#PWR?" H 5800 2700 50  0001 C CNN
+F 1 "+BATT" V 5815 2977 50  0000 L CNN
+F 2 "" H 5800 2850 50  0001 C CNN
+F 3 "" H 5800 2850 50  0001 C CNN
+	1    5800 2850
 	0    -1   -1   0
 $EndComp
@@
 	1    0    0    -1
 $EndComp
-Text Label 5800 3250 2    50   ~ 0
-PWM0
-Text Label 5800 3350 2    50   ~ 0
-PWM1
-Text Label 3500 4150 0    50   ~ 0
-PWM0
-Text Label 3500 4350 0    50   ~ 0
-PWM1
 Text HLabel 5750 6350 0    50   BiDi ~ 0
 USB_D_N
@@
 	0    -1   -1   0
 $EndComp
+NoConn ~ 3500 4150
+NoConn ~ 3500 4350
+$Comp
+L power:GND #PWR?
+U 1 1 5C759BF5
+P 5800 2950
+F 0 "#PWR?" H 5800 2700 50  0001 C CNN
+F 1 "GND" V 5805 2822 50  0000 R CNN
+F 2 "" H 5800 2950 50  0001 C CNN
+F 3 "" H 5800 2950 50  0001 C CNN
+	1    5800 2950
+	0    1    1    0
+$EndComp
+$Comp
+L power:+3.3V #PWR?
+U 1 1 5C75AFA4
+P 5800 2650
+F 0 "#PWR?" H 5800 2500 50  0001 C CNN
+F 1 "+3.3V" V 5815 2778 50  0000 L CNN
+F 2 "" H 5800 2650 50  0001 C CNN
+F 3 "" H 5800 2650 50  0001 C CNN
+	1    5800 2650
+	0    -1   -1   0
+$EndComp

Commit message: +esp32picod4 +fix mounting hole position -ceramic antenna +ufl -spi flash
Parts:
- removed J?: PROG, symbol Connector:Conn_01x05_Female
- removed R16: 47K, Resistor_SMD:R_0402_1005Metric, symbol Device:R
- removed R? (x2): 2K, Resistor_SMD:R_0402_1005Metric, symbol Device:R
- added J?: Ephy, symbol Connector:Conn_01x08_Female
- added J?: CSI, symbol Connector:Conn_01x08_Female
- added J?: AUDIO, symbol Connector:Conn_01x08_Female
- added J?: GPIOA, symbol Connector:Conn_01x08_Female
- added J?: GPIOB, symbol Connector:Conn_01x08_Female
- C32: value 104 -> 100nF
- C33: footprint Capacitor_SMD:C_0603_1608Metric -> Capacitor_SMD:C_0402_1005Metric
- J2: renamed from J?; value Header -> GPIOC
- R10, R11: renamed from R?; value 5.1K -> 2K; footprint (none) -> Resistor_SMD:R_0402_1005Metric
- R17: value 10K -> 2K
- R29: value 47K -> 2K
- TP1, TP2: renamed from TP?; footprint (none) -> TestPoint:TestPoint_Pad_1.0x1.0mm
- TP4: footprint TestPoint:TestPoint_Pad_D1.0mm -> TestPoint:TestPoint_Pad_1.0x1.0mm
- gave numbers to parts that had none: 1
Connections:
- net +BATT is gone; now on net USB_D_P: J2.3 (Pin_3)
- net +3V3: no longer J2.1 (Pin_1)
- net GND: now also J?.3 (Pin_3), J?.3 (Pin_3), J?.6 (Pin_6), J?.6 (Pin_6), J?.8 (Pin_8); no longer J2.2 (Pin_2), J2.4 (Pin_4)
- net HPCOM: now also J?.7 (Pin_7)
- net HPCOMFB: now also J?.6 (Pin_6)
- net USB_D_N: now also J2.2 (Pin_2)
- net USB_ID: now also J2.1 (Pin_1)
- net MICIN1P: now reaches U1.113 (MICIN1P)
- net MICIN1P: now also J?.5 (Pin_5)
- net MICIN1N: now reaches U1.114 (MICIN1N)
- net MICIN1N: now also J?.4 (Pin_4)
- net HBIAS: now reaches U1.119 (HBIAS)
- net HBIAS: now also J?.3 (Pin_3)
- net HPOUTR: now reaches U1.120 (HPOUTR)
- net HPOUTR: now also J?.1 (Pin_1)
- net HPOUTL: now reaches U1.121 (HPOUTL)
- net HPOUTL: now also J?.2 (Pin_2)
- net PE20: now reaches U1.10 (PE20/CSI-FIELD/CSI-MIPI-M-CLK)
- net PE20: now also J?.3 (Pin_3)
- net PF5: now reaches U1.101 (PF5/SDC0/D2)
- net PF5: now also J?.6 (Pin_6)
- net PF4: now reaches U1.102 (PF4/SDC0/D3)
- net PF4: now also J?.5 (Pin_5)
- net PF3: now reaches U1.103 (PF3/SDC0/CMD)
- net PF3: now also J?.4 (Pin_4)
- net PF2: now reaches U1.105 (PF2/SDC0/CLK)
- net PF2: now also J?.3 (Pin_3)
- net PF1: now reaches U1.106 (PF1/SDC0/D0)
- net PF1: now also J?.2 (Pin_2)
- net PF0: now reaches U1.107 (PF0/SDC0/D1)
- net PF0: now also J?.1 (Pin_1)
- net PE19: now reaches U1.11 (PE19/CSI-D15/LCD-D21)
- net PE19: now also J?.4 (Pin_4)
- net LRDAC0: now reaches U1.112 (LRADC0)
- net LRDAC0: now also J2.4 (Pin_4)
- net PG5: now reaches U1.128 (PG5/SDC1/D3)
- net PG5: now also J?.8 (Pin_8)
- net PE18: now reaches U1.13 (PE18/CSI-D14/LCD-D20)
- net PE18: now also J?.5 (Pin_5)
- net PE17: now reaches U1.14 (PE17/CSI-D13/LCD-D19)
- net PE17: now also J?.6 (Pin_6)
- net PE16: now reaches U1.15 (PE16/CSI-D12/LCD-D18)
- net PE16: now also J?.7 (Pin_7)
- net PWM0: now reaches U1.43 (PB4/PWM0)
- net PWM0: now also J?.7 (Pin_7)
- net PWM1: now reaches U1.44 (PB5/PWM1)
- net PWM1: now also J?.8 (Pin_8)
- net PE24: now reaches U1.6 (PE24/LCD-D23)
- net PE24: now also J?.1 (Pin_1)
- net PE23: now reaches U1.7 (PE23/LCD-D22/)
- net PE23: now also J?.2 (Pin_2)
- net MCSI_D0_P: now reaches U1.81 (MCSI-D0P)
- net MCSI_D0_P: now also J?.1 (Pin_1)
- net MCSI_D0_N: now reaches U1.82 (MCSI-D0N)
- net MCSI_D0_N: now also J?.2 (Pin_2)
- net MCSI_D1_P: now reaches U1.83 (MCSI-D1P)
- net MCSI_D1_P: now also J?.4 (Pin_4)
- net MCSI_D1_N: now reaches U1.84 (MCSI-D1N)
- net MCSI_D1_N: now also J?.5 (Pin_5)
- net MCSI_CK_P: now reaches U1.86 (MCSI-CKP)
- net MCSI_CK_P: now also J?.8 (Pin_8)
- net MCSI_CK_N: now reaches U1.87 (MCSI-CKN)
- net MCSI_CK_N: now also J?.7 (Pin_7)
- net EPHY_LINK_LED: now reaches U1.77 (EPHY_LINK_LED)
- net EPHY_LINK_LED: now also J?.7 (Pin_7)
- net EPHY_SPD_LED: now reaches U1.78 (EPHY_SPD_LED)
- net EPHY_SPD_LED: now also J?.8 (Pin_8)
- net EPHY_RX_N: now reaches U1.89 (EPHY_RXN)
- net EPHY_RX_N: now also J?.1 (Pin_1)
- net EPHY_RX_P: now reaches U1.90 (EPHY_RXP)
- net EPHY_RX_P: now also J?.2 (Pin_2)
- net EPHY_TX_N: now reaches U1.91 (EPHY_TXN)
- net EPHY_TX_N: now also J?.4 (Pin_4)
- net EPHY_TX_P: now reaches U1.92 (EPHY_TXP)
- net EPHY_TX_P: now also J?.5 (Pin_5)
- no-connect marks 41 -> 7
Other:
- moved on the sheet: J2, J3, R10, R11
