File: OB_ESP32/esp32.sch (KiCad schematic (older format))
At the start: 16 parts, among them J1 GPIOC, J5 U.FL-R-SMT(01), U3 WS2812-2020, U5 ESP32-PICO-D4

Commit message: mounting hole placement fix, routing allmost done
Parts:
- removed J1: GPIOC, Connector_PinHeader_1.00mm:PinHeader_1x18_P1.00mm_Vertical, symbol Connector:Conn_01x18_Female
- removed J?: Conn_01x24_Female, symbol Connector:Conn_01x24_Female
- removed U3: WS2812-2020, WS2812-2020:LED_WS2812-2020, symbol WS2812-2020:WS2812-2020
- added J1: GPIOC, Connector_PinHeader_1.27mm:PinHeader_1x20_P1.27mm_Vertical, symbol Connector:Conn_01x20_Female
- J5: footprint HRS_U.FL-R-SMT(01) -> U.FL-R-SMT_01_:HRS_U.FL-R-SMT(01)
Connections:
- net labels added: CLK, CMD, IO21, IO27, IO34, SD0, SD1, SD2
- net labels removed: +BATT, IO16, IO42, SENSOR_CAPN, SENSOR_CAPP, WS2812_DI, WS2812_DO
- no-connect marks 10 -> 7
