File: V3S_ESP32_Feather/esp32.sch (KiCad schematic (older format))
At the start: 22 parts, among them J5 U.FL-R-SMT(01), U4 ICM-20948, U5 ESP32-PICO-D4, U7 BMP280

Commit message: Add i2c connector from V3s, fix sd card detection and remove todos
Parts:
- U7: symbol dk_Pressure-Sensors-Transducers:BMP280 -> V3S_ESP32_Feather-rescue:BMP280-dk_Pressure-Sensors-Transducers
Changed lines of the file:
@@
 $EndComp
 $Comp
-L dk_Pressure-Sensors-Transducers:BMP280 U7
+L V3S_ESP32_Feather-rescue:BMP280-dk_Pressure-Sensors-Transducers U7
 U 1 1 5D80F3DE
 P 10000 3350

Commit message: Add more footprint, pcb format done, started component placement
Parts:
- C11, C13, C14, C15, C16: renamed from C?; footprint (none) -> Capacitor_SMD:C_0201_0603Metric
- R7, R8: renamed from R?; footprint (none) -> Resistor_SMD:R_0201_0603Metric
- U9: renamed from U?; footprint BGA16C50P4X4_202X202X67N -> MAX13030EEBET:BGA16C50P4X4_202X202X67N
Changed lines of the file:
@@
 AR Path="/5BC231CB/5D86B8E1" Ref="#PWR?"  Part="1"
 AR Path="/5D86B8E1" Ref="#PWR?"  Part="1"
-AR Path="/5C7A02C5/5D86B8E1" Ref="#PWR?"  Part="1"
-F 0 "#PWR?" H 850 2350 50  0001 C CNN
+AR Path="/5C7A02C5/5D86B8E1" Ref="#PWR0174"  Part="1"
+F 0 "#PWR0174" H 850 2350 50  0001 C CNN
 F 1 "+BATT" H 865 2673 50  0000 C CNN
 F 2 "" H 850 2500 50  0001 C CNN
@@
 $EndComp
 $Comp
-L Device:R R?
+L Device:R R7
 U 1 1 5D86B9DD
 P 850 2650
-F 0 "R?" H 920 2696 50  0000 L CNN
+F 0 "R7" H 920 2696 50  0000 L CNN
 F 1 "R" H 920 2605 50  0000 L CNN
-F 2 "" V 780 2650 50  0001 C CNN
+F 2 "Resistor_SMD:R_0201_0603Metric" V 780 2650 50  0001 C CNN
 F 3 "~" H 850 2650 50  0001 C CNN
 	1    850  2650
@@
 $EndComp
 $Comp
-L Device:R R?
+L Device:R R8
 U 1 1 5D86CE7F
 P 1000 2500
-F 0 "R?" V 793 2500 50  0000 C CNN
+F 0 "R8" V 793 2500 50  0000 C CNN
 F 1 "R" V 884 2500 50  0000 C CNN
-F 2 "" V 930 2500 50  0001 C CNN
+F 2 "Resistor_SMD:R_0201_0603Metric" V 930 2500 50  0001 C CNN
 F 3 "~" H 1000 2500 50  0001 C CNN
 	1    1000 2500
@@
 	1850 2500 1150 2500
 $Comp
-L power:GND #PWR?
+L power:GND #PWR0181
 U 1 1 5D86EA2E
 P 850 2800
-F 0 "#PWR?" H 850 2550 50  0001 C CNN
+F 0 "#PWR0181" H 850 2550 50  0001 C CNN
 F 1 "GND" H 855 2627 50  0000 C CNN
 F 2 "" H 850 2800 50  0001 C CNN
@@
 $EndComp
 $Comp
-L power:GND #PWR?
+L power:GND #PWR0182
 U 1 1 5D86FCC4
 P 10400 3250
-F 0 "#PWR?" H 10400 3000 50  0001 C CNN
+F 0 "#PWR0182" H 10400 3000 50  0001 C CNN
 F 1 "GND" V 10405 3122 50  0000 R CNN
 F 2 "" H 10400 3250 50  0001 C CNN
@@
 IO21
 $Comp
-L power:+3.3V #PWR?
+L power:+3.3V #PWR0183
 U 1 1 5D874BCC
 P 9600 3350
-F 0 "#PWR?" H 9600 3200 50  0001 C CNN
+F 0 "#PWR0183" H 9600 3200 50  0001 C CNN
 F 1 "+3.3V" V 9615 3478 50  0000 L CNN
 F 2 "" H 9600 3350 50  0001 C CNN
@@
 $EndComp
 $Comp
-L power:GND #PWR?
+L power:GND #PWR0184
 U 1 1 5D876B08
 P 10050 3650
-F 0 "#PWR?" H 10050 3400 50  0001 C CNN
+F 0 "#PWR0184" H 10050 3400 50  0001 C CNN
 F 1 "GND" H 10055 3477 50  0000 C CNN
 F 2 "" H 10050 3650 50  0001 C CNN
@@
 	10050 3650 10000 3650
 $Comp
-L power:+3.3V #PWR?
+L power:+3.3V #PWR0185
 U 1 1 5D878D4D
 P 10000 2600
-F 0 "#PWR?" H 10000 2450 50  0001 C CNN
+F 0 "#PWR0185" H 10000 2450 50  0001 C CNN
 F 1 "+3.3V" V 10015 2728 50  0000 L CNN
 F 2 "" H 10000 2600 50  0001 C CNN
@@
 $EndComp
 $Comp
-L Device:C C?
+L Device:C C16
 U 1 1 5D87A246
 P 9850 2800
-F 0 "C?" V 9598 2800 50  0000 C CNN
+F 0 "C16" V 9598 2800 50  0000 C CNN
 F 1 "100nF" V 9689 2800 50  0000 C CNN
-F 2 "" H 9888 2650 50  0001 C CNN
+F 2 "Capacitor_SMD:C_0201_0603Metric" H 9888 2650 50  0001 C CNN
 F 3 "~" H 9850 2800 50  0001 C CNN
 	1    9850 2800
@@
 $EndComp
 $Comp
-L Device:C C?
+L Device:C C15
 U 1 1 5D87DB13
 P 9850 2400
-F 0 "C?" V 9598 2400 50  0000 C CNN
+F 0 "C15" V 9598 2400 50  0000 C CNN
 F 1 "100nF" V 9689 2400 50  0000 C CNN
-F 2 "" H 9888 2250 50  0001 C CNN
+F 2 "Capacitor_SMD:C_0201_0603Metric" H 9888 2250 50  0001 C CNN
 F 3 "~" H 9850 2400 50  0001 C CNN
 	1    9850 2400
@@
 Connection ~ 10000 2800
 $Comp
-L power:GND #PWR?
+L power:GND #PWR0186
 U 1 1 5D881A45
 P 9700 2600
-F 0 "#PWR?" H 9700 2350 50  0001 C CNN
+F 0 "#PWR0186" H 9700 2350 50  0001 C CNN
 F 1 "GND" V 9705 2472 50  0000 R CNN
 F 2 "" H 9700 2600 50  0001 C CNN
@@
 ripple max. 50mVpp
 $Comp
-L Device:C C?
+L Device:C C14
 U 1 1 5D88E1B7
 P 5800 6900
-F 0 "C?" V 5950 6750 50  0000 C CNN
+F 0 "C14" V 5950 6750 50  0000 C CNN
 F 1 "0.1uF" V 5950 7000 50  0000 C CNN
-F 2 "" H 5838 6750 50  0001 C CNN
+F 2 "Capacitor_SMD:C_0201_0603Metric" H 5838 6750 50  0001 C CNN
 F 3 "~" H 5800 6900 50  0001 C CNN
 	1    5800 6900
@@
 $EndComp
 $Comp
-L power:GND #PWR?
+L power:GND #PWR0187
 U 1 1 5D88F7AE
 P 5950 6900
-F 0 "#PWR?" H 5950 6650 50  0001 C CNN
+F 0 "#PWR0187" H 5950 6650 50  0001 C CNN
 F 1 "GND" V 5955 6772 50  0000 R CNN
 F 2 "" H 5950 6900 50  0001 C CNN
@@
 P 5050 5800
 AR Path="/5BC231CB/5D893E3E" Ref="#PWR?"  Part="1"
-AR Path="/5C7A02C5/5D893E3E" Ref="#PWR?"  Part="1"
-F 0 "#PWR?" H 5050 5650 50  0001 C CNN
+AR Path="/5C7A02C5/5D893E3E" Ref="#PWR0188"  Part="1"
+F 0 "#PWR0188" H 5050 5650 50  0001 C CNN
 F 1 "+1V8" V 5050 6000 50  0000 C CNN
 F 2 "" H 5050 5800 50  0001 C CNN
@@
 $EndComp
 $Comp
-L Device:C C?
+L Device:C C13
 U 1 1 5D893F93
 P 4900 6000
-F 0 "C?" V 4648 6000 50  0000 C CNN
+F 0 "C13" V 4648 6000 50  0000 C CNN
 F 1 "1uF" V 4739 6000 50  0000 C CNN
-F 2 "" H 4938 5850 50  0001 C CNN
+F 2 "Capacitor_SMD:C_0201_0603Metric" H 4938 5850 50  0001 C CNN
 F 3 "~" H 4900 6000 50  0001 C CNN
 	1    4900 6000
@@
 $EndComp
 $Comp
-L power:GND #PWR?
+L power:GND #PWR0189
 U 1 1 5D89630A
 P 4750 5800
-F 0 "#PWR?" H 4750 5550 50  0001 C CNN
+F 0 "#PWR0189" H 4750 5550 50  0001 C CNN
 F 1 "GND" V 4755 5672 50  0000 R CNN
 F 2 "" H 4750 5800 50  0001 C CNN
@@
 $EndComp
 $Comp
-L power:GND #PWR?
+L power:GND #PWR0190
 U 1 1 5D897EE9
 P 5150 7400
-F 0 "#PWR?" H 5150 7150 50  0001 C CNN
+F 0 "#PWR0190" H 5150 7150 50  0001 C CNN
 F 1 "GND" H 5155 7227 50  0000 C CNN
 F 2 "" H 5150 7400 50  0001 C CNN
@@
 NoConn ~ 5650 6700
 $Comp
-L Device:C C?
+L Device:C C11
 U 1 1 5D89B9D3
 P 4900 5600
-F 0 "C?" V 4650 5600 50  0000 C CNN
+F 0 "C11" V 4650 5600 50  0000 C CNN
 F 1 "0.1uF" V 4750 5600 50  0000 C CNN
-F 2 "" H 4938 5450 50  0001 C CNN
+F 2 "Capacitor_SMD:C_0201_0603Metric" H 4938 5450 50  0001 C CNN
 F 3 "~" H 4900 5600 50  0001 C CNN
 	1    4900 5600
@@
 ICM_INT
 $Comp
-L power:GND #PWR?
+L power:GND #PWR0191
 U 1 1 5D8A4A86
 P 4650 6900
-F 0 "#PWR?" H 4650 6650 50  0001 C CNN
+F 0 "#PWR0191" H 4650 6650 50  0001 C CNN
 F 1 "GND" V 4655 6772 50  0000 R CNN
 F 2 "" H 4650 6900 50  0001 C CNN
@@
 	5050 5800 5050 6000
 $Comp
-L power:+1V8 #PWR?
+L power:+1V8 #PWR0192
 U 1 1 5D8C24DF
 P 3000 5850
-F 0 "#PWR?" H 3000 5700 50  0001 C CNN
+F 0 "#PWR0192" H 3000 5700 50  0001 C CNN
 F 1 "+1V8" V 3015 5978 50  0000 L CNN
 F 2 "" H 3000 5850 50  0001 C CNN
@@
 $EndComp
 $Comp
-L power:GND #PWR?
+L power:GND #PWR0193
 U 1 1 5D8C4405
 P 3000 7150
-F 0 "#PWR?" H 3000 6900 50  0001 C CNN
+F 0 "#PWR0193" H 3000 6900 50  0001 C CNN
 F 1 "GND" V 3005 7022 50  0000 R CNN
 F 2 "" H 3000 7150 50  0001 C CNN
@@
 ICM_INT1.8
 $Comp
-L MAX13030EEBET:MAX13030EEBET U?
+L MAX13030EEBET:MAX13030EEBET U9
 U 1 1 5D8CAF65
 P 2300 6550
-F 0 "U?" H 2300 7520 50  0000 C CNN
+F 0 "U9" H 2300 7520 50  0000 C CNN
 F 1 "MAX13030EEBET" H 2300 7429 50  0000 C CNN
-F 2 "BGA16C50P4X4_202X202X67N" H 2300 6550 50  0001 L BNN
+F 2 "MAX13030EEBET:BGA16C50P4X4_202X202X67N" H 2300 6550 50  0001 L BNN
 F 3 "UCSP-16 Maxim" H 2300 6550 50  0001 L BNN
 F 4 "Voltage Level Translator 16-Pin UCSP T/R" H 2300 6550 50  0001 L BNN "Champ4"
@@
 NoConn ~ 1600 6950
 $Comp
-L power:+3.3V #PWR?
+L power:+3.3V #PWR0194
 U 1 1 5D8D4D4C
 P 3000 5950
-F 0 "#PWR?" H 3000 5800 50  0001 C CNN
+F 0 "#PWR0194" H 3000 5800 50  0001 C CNN
 F 1 "+3.3V" V 3015 6078 50  0000 L CNN
 F 2 "" H 3000 5950 50  0001 C CNN
@@
 $EndComp
 $Comp
-L power:+3.3V #PWR?
+L power:+3.3V #PWR0195
 U 1 1 5D8D7289
 P 1600 6150
-F 0 "#PWR?" H 1600 6000 50  0001 C CNN
+F 0 "#PWR0195" H 1600 6000 50  0001 C CNN
 F 1 "+3.3V" V 1615 6278 50  0000 L CNN
 F 2 "" H 1600 6150 50  0001 C CNN

Commit message: New component placement, progress on rooting
Connections:
- net labels added: SD2, SD3
- no-connect marks 14 -> 12
Changed lines of the file:
@@
 Text Label 1600 6450 2    50   ~ 0
 CS
-NoConn ~ 3450 2800
-NoConn ~ 3450 2900
 $Comp
 L Device:R R?
@@
 	0    -1   -1   0
 $EndComp
+Text HLabel 3450 2900 2    50   BiDi ~ 0
+SD2
+Text HLabel 3450 2800 2    50   BiDi ~ 0
+SD3
 $EndSCHEMATC

Commit message: Change Max13030 and moove ESP32
Parts:
- removed U9: MAX13030EEBET, MAX13030EEBET:BGA16C50P4X4_202X202X67N, symbol MAX13030EEBET:MAX13030EEBET
- added U9: MAX13030EETE, MAX13035EETET:QFN65P400X400X80-17N, symbol MAX13035EETET:MAX13030EETE
Connections:
- wire segments 21 -> 23
Changed lines of the file:
@@
 Text Label 3450 3500 0    50   ~ 0
 CS
-Text Label 3000 6450 0    50   ~ 0
+Text Label 1300 6600 2    50   ~ 0
 MOSI
-Text Label 3000 6350 0    50   ~ 0
+Text Label 2700 6800 0    50   ~ 0
 MISO
-Text Label 3000 6550 0    50   ~ 0
+Text Label 1300 6700 2    50   ~ 0
 CLK
-Text Label 1600 6450 2    50   ~ 0
+Text Label 2700 6600 0    50   ~ 0
 CS
 $Comp
@@
 L power:+1V8 #PWR0192
 U 1 1 5D8C24DF
-P 3000 5850
-F 0 "#PWR0192" H 3000 5700 50  0001 C CNN
-F 1 "+1V8" V 3015 5978 50  0000 L CNN
-F 2 "" H 3000 5850 50  0001 C CNN
-F 3 "" H 3000 5850 50  0001 C CNN
-	1    3000 5850
+P 2700 5900
+F 0 "#PWR0192" H 2700 5750 50  0001 C CNN
+F 1 "+1V8" V 2715 6028 50  0000 L CNN
+F 2 "" H 2700 5900 50  0001 C CNN
+F 3 "" H 2700 5900 50  0001 C CNN
+	1    2700 5900
 	0    1    1    0
 $EndComp
@@
 L power:GND #PWR0193
 U 1 1 5D8C4405
-P 3000 7150
-F 0 "#PWR0193" H 3000 6900 50  0001 C CNN
-F 1 "GND" V 3005 7022 50  0000 R CNN
-F 2 "" H 3000 7150 50  0001 C CNN
-F 3 "" H 3000 7150 50  0001 C CNN
-	1    3000 7150
-	0    -1   -1   0
-$EndComp
-Text Label 3000 6850 0    50   ~ 0
+P 2700 7450
+F 0 "#PWR0193" H 2700 7200 50  0001 C CNN
+F 1 "GND" V 2705 7322 50  0000 R CNN
+F 2 "" H 2700 7450 50  0001 C CNN
+F 3 "" H 2700 7450 50  0001 C CNN
+	1    2700 7450
+	0    -1   -1   0
+$EndComp
+Text Label 1300 7000 2    50   ~ 0
 MOSI1.8
-Text Label 3000 6750 0    50   ~ 0
+Text Label 2700 7200 0    50   ~ 0
 MISO1.8
-Text Label 3000 6950 0    50   ~ 0
+Text Label 1300 7100 2    50   ~ 0
 CLK1.8
 Text Label 4650 6500 2    50   ~ 0
@@
 Text Label 4650 6600 2    50   ~ 0
 CLK1.8
-Text Label 1600 6850 2    50   ~ 0
+Text Label 2700 7000 0    50   ~ 0
 CS1.8
 Text Label 4650 6700 2    50   ~ 0
 CS1.8
-Text Label 1600 6350 2    50   ~ 0
+Text Label 2700 6700 0    50   ~ 0
 ICM_INT
-Text Label 1600 6750 2    50   ~ 0
+Text Label 2700 7100 0    50   ~ 0
 ICM_INT1.8
-$Comp
-L MAX13030EEBET:MAX13030EEBET U9
-U 1 1 5D8CAF65
-P 2300 6550
-F 0 "U9" H 2300 7520 50  0000 C CNN
-F 1 "MAX13030EEBET" H 2300 7429 50  0000 C CNN
-F 2 "MAX13030EEBET:BGA16C50P4X4_202X202X67N" H 2300 6550 50  0001 L BNN
-F 3 "UCSP-16 Maxim" H 2300 6550 50  0001 L BNN
-F 4 "Voltage Level Translator 16-Pin UCSP T/R" H 2300 6550 50  0001 L BNN "Champ4"
-F 5 "None" H 2300 6550 50  0001 L BNN "Champ5"
-F 6 "MAX13030EEBE+T" H 2300 6550 50  0001 L BNN "Champ6"
-F 7 "Unavailable" H 2300 6550 50  0001 L BNN "Champ7"
-F 8 "Maxim Integrated" H 2300 6550 50  0001 L BNN "Champ8"
-	1    2300 6550
-	1    0    0    -1
-$EndComp
-NoConn ~ 1600 6550
-NoConn ~ 1600 6950
 $Comp
 L power:+3.3V #PWR0194
 U 1 1 5D8D4D4C
-P 3000 5950
-F 0 "#PWR0194" H 3000 5800 50  0001 C CNN
-F 1 "+3.3V" V 3015 6078 50  0000 L CNN
-F 2 "" H 3000 5950 50  0001 C CNN
-F 3 "" H 3000 5950 50  0001 C CNN
-	1    3000 5950
+P 2700 6100
+F 0 "#PWR0194" H 2700 5950 50  0001 C CNN
+F 1 "+3.3V" V 2715 6228 50  0000 L CNN
+F 2 "" H 2700 6100 50  0001 C CNN
+F 3 "" H 2700 6100 50  0001 C CNN
+	1    2700 6100
 	0    1    1    0
 $EndComp
@@
 L power:+3.3V #PWR0195
 U 1 1 5D8D7289
-P 1600 6150
-F 0 "#PWR0195" H 1600 6000 50  0001 C CNN
-F 1 "+3.3V" V 1615 6278 50  0000 L CNN
-F 2 "" H 1600 6150 50  0001 C CNN
-F 3 "" H 1600 6150 50  0001 C CNN
-	1    1600 6150
+P 1300 6300
+F 0 "#PWR0195" H 1300 6150 50  0001 C CNN
+F 1 "+3.3V" V 1315 6428 50  0000 L CNN
+F 2 "" H 1300 6300 50  0001 C CNN
+F 3 "" H 1300 6300 50  0001 C CNN
+	1    1300 6300
 	0    -1   -1   0
 $EndComp
@@
 Text HLabel 3450 2800 2    50   BiDi ~ 0
 SD3
+$Comp
+L MAX13035EETET:MAX13030EETE U9
+U 1 1 5D8C6B10
+P 2000 6700
+F 0 "U9" H 2000 7770 50  0000 C CNN
+F 1 "MAX13030EETE" H 2000 7679 50  0000 C CNN
+F 2 "MAX13035EETET:QFN65P400X400X80-17N" H 2000 6700 50  0001 L BNN
+F 3 "None" H 2000 6700 50  0001 L BNN
+F 4 "Maxim Integrated" H 2000 6700 50  0001 L BNN "Champ4"
+F 5 "Voltage Level Translator 16-Pin TQFN EP" H 2000 6700 50  0001 L BNN "Champ5"
+F 6 "QFN-16 Maxim" H 2000 6700 50  0001 L BNN "Champ6"
+F 7 "Unavailable" H 2000 6700 50  0001 L BNN "Champ7"
+F 8 "MAX13035EETE+" H 2000 6700 50  0001 L BNN "Champ8"
+	1    2000 6700
+	1    0    0    -1
+$EndComp
+Wire Wire Line
+	2700 7400 2700 7450
+Connection ~ 2700 7450
+Wire Wire Line
+	2700 7450 2700 7500
+NoConn ~ 1300 6400
+NoConn ~ 2700 6000
 $EndSCHEMATC

Commit message: last 4 layers version
Parts:
- added J?: I2C, Connector_JST:JST_SH_SM04B-SRSS-TB_1x04-1MP_P1.00mm_Horizontal, symbol Connector:Conn_01x04_Female
- added J?: PWM, Connector_JST:JST_SH_SM10B-SRSS-TB_1x10-1MP_P1.00mm_Horizontal, symbol Connector:Conn_01x10_Female
Connections:
- net labels added: SCL, SDA
Changed lines of the file:
@@
 NoConn ~ 3450 3000
 NoConn ~ 1850 4100
-Text HLabel 1850 2800 0    50   BiDi ~ 0
-IO35
-Text HLabel 1850 2900 0    50   BiDi ~ 0
-IO34
-Text HLabel 1850 3100 0    50   BiDi ~ 0
-IO33
-Text HLabel 1850 3200 0    50   BiDi ~ 0
-IO32
-Text HLabel 1850 3300 0    50   BiDi ~ 0
-IO27
-Text HLabel 1850 3400 0    50   BiDi ~ 0
-IO26
-Text HLabel 1850 3500 0    50   BiDi ~ 0
-IO25
-Text HLabel 1850 3700 0    50   BiDi ~ 0
-IO22
-Text HLabel 1850 3800 0    50   BiDi ~ 0
-IO21
-Text HLabel 1850 2600 0    50   BiDi ~ 0
-SENSOR_VN
 Wire Wire Line
 	3450 2500 4000 2500
@@
 NoConn ~ 1300 6400
 NoConn ~ 2700 6000
+Text Label 8450 5550 2    50   ~ 0
+IO33
+Text Label 8450 5450 2    50   ~ 0
+IO32
+Text Label 8450 5850 2    50   ~ 0
+IO27
+Text Label 8450 5750 2    50   ~ 0
+IO26
+Text Label 8450 5650 2    50   ~ 0
+IO25
+$Comp
+L power:GND #PWR?
+U 1 1 5D90AFA4
+P 8450 5950
+AR Path="/5D90AFA4" Ref="#PWR?"  Part="1"
+AR Path="/5C7A02C5/5D90AFA4" Ref="#PWR?"  Part="1"
+F 0 "#PWR?" H 8450 5700 50  0001 C CNN
+F 1 "GND" V 8450 5700 50  0000 C CNN
+F 2 "" H 8450 5950 50  0001 C CNN
+F 3 "" H 8450 5950 50  0001 C CNN
+	1    8450 5950
+	0    1    1    0
+$EndComp
+Text Label 8450 5250 2    50   ~ 0
+IO34
+Text Label 9450 5550 2    50   ~ 0
+SDA
+Text Label 9450 5650 2    50   ~ 0
+SCL
+$Comp
+L Connector:Conn_01x04_Female J?
+U 1 1 5D90AFAD
+P 9650 5550
+AR Path="/5D90AFAD" Ref="J?"  Part="1"
+AR Path="/5C7A02C5/5D90AFAD" Ref="J?"  Part="1"
+F 0 "J?" H 9678 5526 50  0000 L CNN
+F 1 "I2C" H 9678 5435 50  0000 L CNN
+F 2 "Connector_JST:JST_SH_SM04B-SRSS-TB_1x04-1MP_P1.00mm_Horizontal" H 9650 5550 50  0001 C CNN
+F 3 "~" H 9650 5550 50  0001 C CNN
+	1    9650 5550
+	1    0    0    -1
+$EndComp
+$Comp
+L power:GND #PWR?
+U 1 1 5D90AFB3
+P 9450 5450
+AR Path="/5D90AFB3" Ref="#PWR?"  Part="1"
+AR Path="/5C7A02C5/5D90AFB3" Ref="#PWR?"  Part="1"
+F 0 "#PWR?" H 9450 5200 50  0001 C CNN
+F 1 "GND" H 9455 5277 50  0000 C CNN
+F 2 "" H 9450 5450 50  0001 C CNN
+F 3 "" H 9450 5450 50  0001 C CNN
+	1    9450 5450
+	-1   0    0    1
+$EndComp
+$Comp
+L power:+3.3V #PWR?
+U 1 1 5D90AFB9
+P 9450 5750
+AR Path="/5D90AFB9" Ref="#PWR?"  Part="1"
+AR Path="/5C7A02C5/5D90AFB9" Ref="#PWR?"  Part="1"
+F 0 "#PWR?" H 9450 5600 50  0001 C CNN
+F 1 "+3.3V" V 9465 5878 50  0000 L CNN
+F 2 "" H 9450 5750 50  0001 C CNN
+F 3 "" H 9450 5750 50  0001 C CNN
+	1    9450 5750
+	0    -1   -1   0
+$EndComp
+$Comp
+L power:+BATT #PWR?
+U 1 1 5D90AFBF
+P 8450 5050
+AR Path="/5BC231CB/5D90AFBF" Ref="#PWR?"  Part="1"
+AR Path="/5D90AFBF" Ref="#PWR?"  Part="1"
+AR Path="/5C7A02C5/5D90AFBF" Ref="#PWR?"  Part="1"
+F 0 "#PWR?" H 8450 4900 50  0001 C CNN
+F 1 "+BATT" V 8450 5300 50  0000 C CNN
+F 2 "" H 8450 5050 50  0001 C CNN
+F 3 "" H 8450 5050 50  0001 C CNN
+	1    8450 5050
+	0    -1   -1   0
+$EndComp
+Text Label 8450 5350 2    50   ~ 0
+IO35
+$Comp
+L Connector:Conn_01x10_Female J?
+U 1 1 5D90AFC6
+P 8650 5450
+AR Path="/5D90AFC6" Ref="J?"  Part="1"
+AR Path="/5C7A02C5/5D90AFC6" Ref="J?"  Part="1"
+F 0 "J?" H 8678 5426 50  0000 L CNN
+F 1 "PWM" H 8678 5335 50  0000 L CNN
+F 2 "Connector_JST:JST_SH_SM10B-SRSS-TB_1x10-1MP_P1.00mm_Horizontal" H 8650 5450 50  0001 C CNN
+F 3 "~" H 8650 5450 50  0001 C CNN
+	1    8650 5450
+	1    0    0    -1
+$EndComp
+Text Label 8450 5150 2    50   ~ 0
+SENSOR_VN
+Text Label 1850 3100 2    50   ~ 0
+IO33
+Text Label 1850 3200 2    50   ~ 0
+IO32
+Text Label 1850 3300 2    50   ~ 0
+IO27
+Text Label 1850 3400 2    50   ~ 0
+IO26
+Text Label 1850 3500 2    50   ~ 0
+IO25
+Text Label 1850 2900 2    50   ~ 0
+IO34
+Text Label 1850 2800 2    50   ~ 0
+IO35
+Text Label 1850 2600 2    50   ~ 0
+SENSOR_VN
+Text Label 1850 3700 2    50   ~ 0
+SDA
+Text Label 1850 3800 2    50   ~ 0
+SCL
 $EndSCHEMATC

Commit message: replace 3 ldo by 1, replace icm by mpu and progress on 2 layer
Parts:
- removed U4: ICM-20948, Sensor_Motion:InvenSense_QFN-24_3x3mm_P0.4mm, symbol Sensor_Motion:ICM-20948
- removed U9: MAX13030EETE, MAX13035EETET:QFN65P400X400X80-17N, symbol MAX13035EETET:MAX13030EETE
- added U3: MPU-9250_Obsolete, digikey-footprints:QFN-24-1EP_3x3mm, symbol dk_Motion-Sensors-IMUs-Inertial-Measurement-Units:MPU-9250_Obsolete
- C11: value 0.1uF -> 10nF
- C13: value 1uF -> 0.1uF
- gave numbers to parts that had none: 2
Connections:
- net labels removed: +1V8, CLK1.8, CS1.8, ICM_INT1.8, IO21, IO22, MISO1.8, MOSI1.8
- wire segments 23 -> 24
- no-connect marks 12 -> 10
Other:
- moved on the sheet: C11, C13, C14

Commit message: almost everything is routed !
Parts:
- U3: symbol dk_Motion-Sensors-IMUs-Inertial-Measurement-Units:MPU-9250_Obsolete -> V3S_ESP32_Feather-rescue:MPU-9250_Obsolete-dk_Motion-Sensors-IMUs-Inertial-Measurement-Units
Changed lines of the file:
@@
 $EndComp
 $Comp
-L dk_Motion-Sensors-IMUs-Inertial-Measurement-Units:MPU-9250_Obsolete U3
+L V3S_ESP32_Feather-rescue:MPU-9250_Obsolete-dk_Motion-Sensors-IMUs-Inertial-Measurement-Units U3
 U 1 1 5D95AEEF
 P 3050 6050
+AR Path="/5D95AEEF" Ref="U3"  Part="1"
+AR Path="/5C7A02C5/5D95AEEF" Ref="U3"  Part="1"
 F 0 "U3" H 3600 5650 60  0000 C CNN
 F 1 "MPU-9250_Obsolete" H 3650 5550 60  0000 C CNN
