File: V3S_ESP32_Feather/power.sch (KiCad schematic (older format))
At the start: 36 parts, among them Q1 S8050(SOT-23), U1 V3S

Commit message: Add more footprint, pcb format done, started component placement
Parts:
- C10, C3, C6, C7, C8: renamed from C?; footprint (none) -> Capacitor_SMD:C_0201_0603Metric
- C2: footprint (none) -> Capacitor_SMD:C_0402_1005Metric
- C43, C44, C55, C56: footprint Capacitor_SMD:C_0201_0603Metric -> Capacitor_SMD:C_0402_1005Metric
- C5, C9: renamed from C?; footprint (none) -> Capacitor_SMD:C_0402_1005Metric
- C61, C63, C64, C65: footprint Capacitor_SMD:C_0402_1005Metric -> Capacitor_SMD:C_0201_0603Metric
- D1: footprint (none) -> Resistor_SMD:R_0603_1608Metric
- TP1: footprint Connector_PinSocket_2.54mm:PinSocket_1x01_P2.54mm_Vertical -> TestPoint:TestPoint_Pad_D1.0mm
- gave numbers to parts that had none: 4

Commit message: New component placement, progress on rooting
Parts:
- removed C2: 10uF, Capacitor_SMD:C_0402_1005Metric, symbol Device:C
- removed Q1: S8050(SOT-23), Package_TO_SOT_SMD:SOT-23, symbol V3S_ESP32_Feather-rescue:SMD-TRANSISTORS-NPN-25V-500MW-S8050(SOT-23)-SMD-TRANSI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
- removed R2: 100K, Resistor_SMD:R_0201_0603Metric, symbol Device:R
- removed TP1: PWR_SRC, TestPoint:TestPoint_Pad_D1.0mm, symbol Connector:TestPoint
Connections:
- wire segments 78 -> 74
Other:
- moved on the sheet: D1, R1
Changed lines of the file:
@@
-$EndComp
-$Comp
-L V3S_ESP32_Feather-rescue:SMD-TRANSISTORS-NPN-25V-500MW-S8050(SOT-23)-SMD-TRANSISTORS-NPN-25V-500MW-S8050_SOT-23_ Q1
-U 1 1 5D33707E
-P 8000 3950
-F 0 "Q1" H 8100 4000 50  0000 L CNN
-F 1 "S8050(SOT-23)" H 7700 4550 50  0000 L CNN
-F 2 "Package_TO_SOT_SMD:SOT-23" H 8000 3950 50  0001 L BNN
-F 3 "" H 8000 3950 50  0001 L BNN
-F 4 "SOT-23-3 JCET" H 8000 3950 50  0001 L BNN "Field4"
-F 5 "S8050" H 8000 3950 50  0001 L BNN "Field5"
-F 6 "Unavailable" H 8000 3950 50  0001 L BNN "Field6"
-F 7 "None" H 8000 3950 50  0001 L BNN "Field7"
-F 8 "JCET" H 8000 3950 50  0001 L BNN "Field8"
-	1    8000 3950
-	1    0    0    -1
-$EndComp
-$Comp
-L Device:R R2
-U 1 1 5D338373
-P 7500 4100
-F 0 "R2" H 7570 4146 50  0000 L CNN
-F 1 "100K" H 7570 4055 50  0000 L CNN
-F 2 "Resistor_SMD:R_0201_0603Metric" V 7430 4100 50  0001 C CNN
-F 3 "~" H 7500 4100 50  0001 C CNN
-	1    7500 4100
-	1    0    0    -1
 $EndComp
 $Comp
 L Device:R R1
 U 1 1 5D339AF0
-P 7500 3800
-F 0 "R1" H 7570 3846 50  0000 L CNN
-F 1 "0" H 7570 3755 50  0000 L CNN
-F 2 "Resistor_SMD:R_0201_0603Metric" V 7430 3800 50  0001 C CNN
-F 3 "~" H 7500 3800 50  0001 C CNN
-	1    7500 3800
-	1    0    0    -1
-$EndComp
-$Comp
-L Connector:TestPoint TP1
-U 1 1 5D33A93A
-P 7500 3950
-F 0 "TP1" V 7300 4350 50  0000 C CNN
-F 1 "PWR_SRC" V 7400 4250 50  0000 C CNN
-F 2 "TestPoint:TestPoint_Pad_D1.0mm" H 7700 3950 50  0001 C CNN
-F 3 "~" H 7700 3950 50  0001 C CNN
-	1    7500 3950
-	0    -1   1    0
-$EndComp
-Connection ~ 7500 3950
-$Comp
-L power:GND #PWR0119
-U 1 1 5D33F3EC
-P 7500 4250
-F 0 "#PWR0119" H 7500 4000 50  0001 C CNN
-F 1 "GND" H 7505 4077 50  0000 C CNN
-F 2 "" H 7500 4250 50  0001 C CNN
-F 3 "" H 7500 4250 50  0001 C CNN
-	1    7500 4250
-	1    0    0    -1
+P 7450 3250
+F 0 "R1" H 7520 3296 50  0000 L CNN
+F 1 "0" H 7520 3205 50  0000 L CNN
+F 2 "Resistor_SMD:R_0201_0603Metric" V 7380 3250 50  0001 C CNN
+F 3 "~" H 7450 3250 50  0001 C CNN
+	1    7450 3250
+	0    1    1    0
 $EndComp
 $Comp
 L Device:D D1
 U 1 1 5D3450C1
-P 7950 4150
-F 0 "D1" H 7950 4250 50  0000 C CNN
-F 1 "D" H 7950 4350 50  0000 C CNN
-F 2 "Resistor_SMD:R_0603_1608Metric" H 7950 4150 50  0001 C CNN
-F 3 "~" H 7950 4150 50  0001 C CNN
-	1    7950 4150
+P 7750 3250
+F 0 "D1" H 7750 3350 50  0000 C CNN
+F 1 "D" H 7750 3450 50  0000 C CNN
+F 2 "Resistor_SMD:R_0603_1608Metric" H 7750 3250 50  0001 C CNN
+F 3 "~" H 7750 3250 50  0001 C CNN
+	1    7750 3250
 	-1   0    0    1
 $EndComp
-Wire Wire Line
-	7800 3950 7800 4150
-Wire Wire Line
-	7500 3950 7800 3950
-Wire Wire Line
-	7800 3950 7900 3950
-Connection ~ 7800 3950
-$Comp
-L Device:C C2
-U 1 1 5D349831
-P 8100 4400
-F 0 "C2" H 8215 4446 50  0000 L CNN
-F 1 "10uF" H 8215 4355 50  0000 L CNN
-F 2 "Capacitor_SMD:C_0402_1005Metric" H 8138 4250 50  0001 C CNN
-F 3 "~" H 8100 4400 50  0001 C CNN
-	1    8100 4400
-	1    0    0    -1
-$EndComp
-Wire Wire Line
-	8100 4250 8100 4150
-Connection ~ 8100 4150
 $Comp
 L power:+BATT #PWR0120
 U 1 1 5D34BFCB
-P 8100 3750
-F 0 "#PWR0120" H 8100 3600 50  0001 C CNN
-F 1 "+BATT" H 8115 3923 50  0000 C CNN
-F 2 "" H 8100 3750 50  0001 C CNN
-F 3 "" H 8100 3750 50  0001 C CNN
-	1    8100 3750
-	1    0    0    -1
-$EndComp
-$Comp
-L power:GND #PWR0121
-U 1 1 5D34CD04
-P 8100 4550
-F 0 "#PWR0121" H 8100 4300 50  0001 C CNN
-F 1 "GND" H 8105 4377 50  0000 C CNN
-F 2 "" H 8100 4550 50  0001 C CNN
-F 3 "" H 8100 4550 50  0001 C CNN
-	1    8100 4550
-	1    0    0    -1
-$EndComp
-Wire Wire Line
-	8100 4150 8650 4150
+P 7900 3250
+F 0 "#PWR0120" H 7900 3100 50  0001 C CNN
+F 1 "+BATT" H 7915 3423 50  0000 C CNN
+F 2 "" H 7900 3250 50  0001 C CNN
+F 3 "" H 7900 3250 50  0001 C CNN
+	1    7900 3250
+	1    0    0    -1
+$EndComp
 $Comp
 L power:VBUS #PWR?
 U 1 1 5D84F1B1
-P 7500 3650
+P 7300 3250
 AR Path="/5D84F1B1" Ref="#PWR?"  Part="1"
 AR Path="/5BC231CB/5D84F1B1" Ref="#PWR0149"  Part="1"
-F 0 "#PWR0149" H 7500 3500 50  0001 C CNN
-F 1 "VBUS" V 7515 3778 50  0000 L CNN
-F 2 "" H 7500 3650 50  0001 C CNN
-F 3 "" H 7500 3650 50  0001 C CNN
-	1    7500 3650
-	1    0    0    -1
+F 0 "#PWR0149" H 7300 3100 50  0001 C CNN
+F 1 "VBUS" V 7315 3378 50  0000 L CNN
+F 2 "" H 7300 3250 50  0001 C CNN
+F 3 "" H 7300 3250 50  0001 C CNN
+	1    7300 3250
+	0    -1   -1   0
 $EndComp
 $Comp
@@
 $EndComp
 Connection ~ 10450 4000
-Text Label 8650 4150 0    50   ~ 0
+Text Label 8050 3250 0    50   ~ 0
 VIN
 Text Label 9300 4000 2    50   ~ 0
@@
 Wire Wire Line
 	9900 5400 9900 5600
+Wire Wire Line
+	7900 3250 8050 3250
+Connection ~ 7900 3250
 $EndSCHEMATC

Commit message: replace 3 ldo by 1, replace icm by mpu and progress on 2 layer
Parts:
- removed R1: 0, Resistor_SMD:R_0201_0603Metric, symbol Device:R
- removed U2: MIC5504-1.2YM5, Package_TO_SOT_SMD:SOT-23-5, symbol Regulator_Linear:MIC5504-1.2YM5
- removed U3: MIC5501-3.0YM5, Package_TO_SOT_SMD:SOT-23-5, symbol Regulator_Linear:MIC5501-3.0YM5
- removed U8: MIC5504-1.8YM5, Package_TO_SOT_SMD:SOT-23-5, symbol Regulator_Linear:MIC5504-1.8YM5
- added C2: 1uF, Capacitor_SMD:C_0201_0603Metric, symbol Device:C
- added D2: D, Resistor_SMD:R_0603_1608Metric, symbol Device:D
- added U2: ADP322ACPZ-145-R7, QFN50P300X300X90-17N:QFN50P300X300X90-17N, symbol 2019-06-13_12-28-51:ADP322ACPZ-145-R7
Connections:
- wire segments 74 -> 77
Other:
- moved on the sheet: C10, C3, C6, D1

Commit message: almost everything is routed !
Parts:
- added C17: 10uF, Capacitor_SMD:C_0201_0603Metric, symbol Device:C
Connections:
- net labels removed: VCC_PE
- wire segments 77 -> 81
Other:
- moved on the sheet: C61
Changed lines of the file:
@@
 	1400 5500 1400 5700
 Connection ~ 1400 5500
-Text Label 1250 4800 2    50   ~ 0
-VCC_PE
-Wire Wire Line
-	1250 4800 1400 4800
-Wire Wire Line
-	1400 4800 1400 4700
-Wire Wire Line
-	1400 4800 1400 4900
-Connection ~ 1400 4800
 $Comp
 L power:+1V2 #PWR0112
@@
 U 1 1 5BD06484
 P 2300 1050
-F 0 "C54" H 2415 1096 50  0000 L CNN
-F 1 "100nF" H 2100 850 50  0000 L CNN
+F 0 "C54" H 2100 1150 50  0000 L CNN
+F 1 "100nF" H 2050 950 50  0000 L CNN
 F 2 "Capacitor_SMD:C_0402_1005Metric" H 2338 900 50  0001 C CNN
 F 3 "~" H 2300 1050 50  0001 C CNN
@@
 U 1 1 5BD0648B
 P 2650 1050
-F 0 "C56" H 2765 1096 50  0000 L CNN
-F 1 "10uF" H 2750 850 50  0000 L CNN
+F 0 "C56" H 2700 1150 50  0000 L CNN
+F 1 "10uF" H 2700 950 50  0000 L CNN
 F 2 "Capacitor_SMD:C_0402_1005Metric" H 2688 900 50  0001 C CNN
 F 3 "~" H 2650 1050 50  0001 C CNN
@@
 L Device:C C61
 U 1 1 5BDFB49E
-P 3450 1050
-F 0 "C61" V 3198 1050 50  0000 C CNN
-F 1 "100nF" V 3289 1050 50  0000 C CNN
-F 2 "Capacitor_SMD:C_0201_0603Metric" H 3488 900 50  0001 C CNN
-F 3 "~" H 3450 1050 50  0001 C CNN
-	1    3450 1050
-	0    1    1    0
+P 3650 1050
+F 0 "C61" H 3500 950 50  0000 C CNN
+F 1 "100nF" H 3500 1150 50  0000 C CNN
+F 2 "Capacitor_SMD:C_0201_0603Metric" H 3688 900 50  0001 C CNN
+F 3 "~" H 3650 1050 50  0001 C CNN
+	1    3650 1050
+	-1   0    0    1
 $EndComp
 $Comp
 L OB-rescue:GND-OLIMEX_Power #PWR0214
 U 1 1 5BE02A91
-P 3600 1050
-F 0 "#PWR0214" H 3600 800 50  0001 C CNN
-F 1 "GND" V 3605 922 50  0000 R CNN
-F 2 "" H 3600 1050 60  0000 C CNN
-F 3 "" H 3600 1050 60  0000 C CNN
-	1    3600 1050
-	0    -1   -1   0
+P 3450 1200
+F 0 "#PWR0214" H 3450 950 50  0001 C CNN
+F 1 "GND" V 3455 1072 50  0000 R CNN
+F 2 "" H 3450 1200 60  0000 C CNN
+F 3 "" H 3450 1200 60  0000 C CNN
+	1    3450 1200
+	1    0    0    -1
 $EndComp
 $Comp
@@
 Connection ~ 2300 900
 $Comp
-L power:+3.3V #PWR0114
-U 1 1 5D8CAE62
-P 3300 1050
-F 0 "#PWR0114" H 3300 900 50  0001 C CNN
-F 1 "+3.3V" V 3315 1178 50  0000 L CNN
-F 2 "" H 3300 1050 50  0001 C CNN
-F 3 "" H 3300 1050 50  0001 C CNN
-	1    3300 1050
-	0    -1   -1   0
-$EndComp
-$Comp
 L power:+3.3V #PWR0122
 U 1 1 5D8CD0D3
@@
 	0    -1   -1   0
 $EndComp
+$Comp
+L power:+3V0 #PWR0114
+U 1 1 5D91094D
+P 3450 900
+F 0 "#PWR0114" H 3450 750 50  0001 C CNN
+F 1 "+3V0" H 3350 1050 50  0000 L CNN
+F 2 "" H 3450 900 50  0001 C CNN
+F 3 "" H 3450 900 50  0001 C CNN
+	1    3450 900
+	1    0    0    -1
+$EndComp
+$Comp
+L power:+3.3V #PWR0144
+U 1 1 5D947F4E
+P 1000 4800
+F 0 "#PWR0144" H 1000 4650 50  0001 C CNN
+F 1 "+3.3V" H 1015 4973 50  0000 C CNN
+F 2 "" H 1000 4800 50  0001 C CNN
+F 3 "" H 1000 4800 50  0001 C CNN
+	1    1000 4800
+	1    0    0    -1
+$EndComp
+Wire Wire Line
+	1400 4700 1400 4800
+Wire Wire Line
+	1400 4800 1000 4800
+Connection ~ 1400 4800
+Wire Wire Line
+	1400 4800 1400 4900
+$Comp
+L Device:C C17
+U 1 1 5D951C71
+P 3250 1050
+F 0 "C17" H 3350 950 50  0000 C CNN
+F 1 "10uF" H 3400 1150 50  0000 C CNN
+F 2 "Capacitor_SMD:C_0201_0603Metric" H 3288 900 50  0001 C CNN
+F 3 "~" H 3250 1050 50  0001 C CNN
+	1    3250 1050
+	-1   0    0    1
+$EndComp
+Wire Wire Line
+	3250 900  3450 900
+Connection ~ 3450 900
+Wire Wire Line
+	3450 900  3650 900
+Wire Wire Line
+	3250 1200 3450 1200
+Connection ~ 3450 1200
+Wire Wire Line
+	3450 1200 3650 1200
 $EndSCHEMATC

Commit message: routing done, started filling bom
Parts:
- C17: footprint Capacitor_SMD:C_0201_0603Metric -> Capacitor_SMD:C_0402_1005Metric
- C48, C49, C54: footprint Capacitor_SMD:C_0402_1005Metric -> Capacitor_SMD:C_0201_0603Metric
Changed lines of the file:
@@
 F 0 "C48" H 5015 1096 50  0000 L CNN
 F 1 "100nF" H 5000 850 50  0000 L CNN
-F 2 "Capacitor_SMD:C_0402_1005Metric" H 4938 900 50  0001 C CNN
+F 2 "Capacitor_SMD:C_0201_0603Metric" H 4938 900 50  0001 C CNN
 F 3 "~" H 4900 1050 50  0001 C CNN
 	1    4900 1050
@@
 F 0 "C49" H 7565 1096 50  0000 L CNN
 F 1 "100nF" H 7550 850 50  0000 L CNN
-F 2 "Capacitor_SMD:C_0402_1005Metric" H 7488 900 50  0001 C CNN
+F 2 "Capacitor_SMD:C_0201_0603Metric" H 7488 900 50  0001 C CNN
 F 3 "~" H 7450 1050 50  0001 C CNN
 	1    7450 1050
@@
 F 0 "C54" H 2100 1150 50  0000 L CNN
 F 1 "100nF" H 2050 950 50  0000 L CNN
-F 2 "Capacitor_SMD:C_0402_1005Metric" H 2338 900 50  0001 C CNN
+F 2 "Capacitor_SMD:C_0201_0603Metric" H 2338 900 50  0001 C CNN
 F 3 "~" H 2300 1050 50  0001 C CNN
 	1    2300 1050
@@
 F 0 "C17" H 3350 950 50  0000 C CNN
 F 1 "10uF" H 3400 1150 50  0000 C CNN
-F 2 "Capacitor_SMD:C_0201_0603Metric" H 3288 900 50  0001 C CNN
+F 2 "Capacitor_SMD:C_0402_1005Metric" H 3288 900 50  0001 C CNN
 F 3 "~" H 3250 1050 50  0001 C CNN
 	1    3250 1050
