File: V3S_ESP32_Feather/power.sch (KiCad schematic (older format))
At the start: 32 parts, among them U1 V3S, U2 ADP322ACPZ-145-R7, U6 LT1963AxST-3.3

Commit message: fix d1, d2 package
Parts:
- D1, D2: footprint Resistor_SMD:R_0603_1608Metric -> Diode_SMD:D_0201_0603Metric
Changed lines of the file:
@@
 F 0 "D1" H 7450 3350 50  0000 C CNN
 F 1 "D" H 7450 3450 50  0000 C CNN
-F 2 "Resistor_SMD:R_0603_1608Metric" H 7450 3250 50  0001 C CNN
+F 2 "Diode_SMD:D_0201_0603Metric" H 7450 3250 50  0001 C CNN
 F 3 "~" H 7450 3250 50  0001 C CNN
 	1    7450 3250
@@
 F 0 "D2" H 7450 3050 50  0000 C CNN
 F 1 "D" H 7450 3150 50  0000 C CNN
-F 2 "Resistor_SMD:R_0603_1608Metric" H 7450 2950 50  0001 C CNN
+F 2 "Diode_SMD:D_0201_0603Metric" H 7450 2950 50  0001 C CNN
 F 3 "~" H 7450 2950 50  0001 C CNN
 	1    7450 2950

Commit message: fix component packages
Parts:
- C17, C43, C44, C5, C55, C56, C9: footprint Capacitor_SMD:C_0402_1005Metric -> Capacitor_SMD:C_0805_2012Metric
Changed lines of the file:
@@
 F 0 "C44" H 4315 1096 50  0000 L CNN
 F 1 "10uF" H 4300 850 50  0000 L CNN
-F 2 "Capacitor_SMD:C_0402_1005Metric" H 4238 900 50  0001 C CNN
+F 2 "Capacitor_SMD:C_0805_2012Metric" H 4238 900 50  0001 C CNN
 F 3 "~" H 4200 1050 50  0001 C CNN
 	1    4200 1050
@@
 F 0 "C43" H 6815 1096 50  0000 L CNN
 F 1 "10uF" H 6800 850 50  0000 L CNN
-F 2 "Capacitor_SMD:C_0402_1005Metric" H 6738 900 50  0001 C CNN
+F 2 "Capacitor_SMD:C_0805_2012Metric" H 6738 900 50  0001 C CNN
 F 3 "~" H 6700 1050 50  0001 C CNN
 	1    6700 1050
@@
 F 0 "C55" H 5565 1096 50  0000 L CNN
 F 1 "10uF" H 5550 850 50  0000 L CNN
-F 2 "Capacitor_SMD:C_0402_1005Metric" H 5488 900 50  0001 C CNN
+F 2 "Capacitor_SMD:C_0805_2012Metric" H 5488 900 50  0001 C CNN
 F 3 "~" H 5450 1050 50  0001 C CNN
 	1    5450 1050
@@
 F 0 "C56" H 2700 1150 50  0000 L CNN
 F 1 "10uF" H 2700 950 50  0000 L CNN
-F 2 "Capacitor_SMD:C_0402_1005Metric" H 2688 900 50  0001 C CNN
+F 2 "Capacitor_SMD:C_0805_2012Metric" H 2688 900 50  0001 C CNN
 F 3 "~" H 2650 1050 50  0001 C CNN
 	1    2650 1050
@@
 F 0 "C5" H 9415 4196 50  0000 L CNN
 F 1 "10uF" H 9415 4105 50  0000 L CNN
-F 2 "Capacitor_SMD:C_0402_1005Metric" H 9338 4000 50  0001 C CNN
+F 2 "Capacitor_SMD:C_0805_2012Metric" H 9338 4000 50  0001 C CNN
 F 3 "~" H 9300 4150 50  0001 C CNN
 	1    9300 4150
@@
 F 0 "C9" H 10565 4196 50  0000 L CNN
 F 1 "10uF" H 10565 4105 50  0000 L CNN
-F 2 "Capacitor_SMD:C_0402_1005Metric" H 10488 4000 50  0001 C CNN
+F 2 "Capacitor_SMD:C_0805_2012Metric" H 10488 4000 50  0001 C CNN
 F 3 "~" H 10450 4150 50  0001 C CNN
 	1    10450 4150
@@
 F 0 "C17" H 3350 950 50  0000 C CNN
 F 1 "10uF" H 3400 1150 50  0000 C CNN
-F 2 "Capacitor_SMD:C_0402_1005Metric" H 3288 900 50  0001 C CNN
+F 2 "Capacitor_SMD:C_0805_2012Metric" H 3288 900 50  0001 C CNN
 F 3 "~" H 3250 1050 50  0001 C CNN
 	1    3250 1050
