File: FPGA_ESP32/_autosave-FPGA_ESP32.kicad_pcb (KiCad board)
At the start: 2 copper layers, 20 x 20 mm, 41 parts, among them J1 Conn_01x18_Female, J2 CAM, J3 Conn_01x18_Female, J4 Conn_01x18_Female, U1 LFE5UM-25F-7MG285C, U10 GD25Q16CEIGR, U2 ESP32-PICO-D4, U3 TMUX1574, U4 W956D6KBKX, U6 W956D6KBKX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

Commit message: FPGA_ESP32 : add camera, change header position
Parts:
- added C10: 1uF, Capacitor_SMD:C_0402_1005Metric, F.Cu at (119.0, 2.10)
- added C11: 0.1uF, Capacitor_SMD:C_0402_1005Metric, F.Cu at (119.0, 4.09)
- added C12: C, Capacitor_SMD:C_0402_1005Metric, F.Cu at (121.9, 2.10)
- added C13: C, Capacitor_SMD:C_0402_1005Metric, F.Cu at (121.9, 4.09)
- added C8: 0.1uF, Capacitor_SMD:C_0402_1005Metric, F.Cu at (116.1, 2.10)
- added C9: 0.1uF, Capacitor_SMD:C_0402_1005Metric, F.Cu at (116.1, 4.09)
- added H1: MountingHole_Pad, MountingHole:MountingHole_2.2mm_M2_Pad_Via, F.Cu at (93.5, 4.08)
- added H2: MountingHole_Pad, MountingHole:MountingHole_2.2mm_M2_Pad_Via, F.Cu at (93.5, 10.0)
- added H3: MountingHole_Pad, MountingHole:MountingHole_2.2mm_M2_Pad_Via, F.Cu at (99.4, 4.08)
- added H4: MountingHole_Pad, MountingHole:MountingHole_2.2mm_M2_Pad, F.Cu at (99.4, 10.0)
Connections:
- net Net-(U2-Pad9) renamed EN
- net Net-(U3-Pad13) renamed /WIFI, BT, RT/SPI_EN
- net Net-(U3-Pad15) renamed /WIFI, BT, RT/SEL
- U2 pad 1: Net-(U2-Pad1) -> VIO
- U2 pad 19: Net-(U2-Pad19) -> VIO
- U2 pad 3: Net-(U2-Pad3) -> VIO
- U2 pad 37: Net-(U2-Pad37) -> VIO
- U2 pad 4: Net-(U2-Pad3) -> VIO
- U2 pad 43: Net-(U2-Pad1) -> VIO
- U2 pad 46: Net-(U2-Pad1) -> VIO
- U3 pad 14: Net-(U3-Pad14) -> VIO
- U3 pad 6: Net-(U3-Pad6) -> GND
