File: FPGA_ESP32/FPGA_ESP32.sch (KiCad schematic (older format))
At the start: 13 parts, among them J1 Conn_01x14_Female, J3 Conn_01x14_Female, J4 Conn_01x14_Female, J5 Conn_01x14_Female, U1 LFE5UM-25F-7MG285C

Commit message: FPGA_ESP32 : esp32 enable circuit, flash done, more doc, TODO power !
Parts:
- removed unit 10 of U1
Connections:
- net labels added: IO27
- net labels removed: +1V1, +2V5
- wire segments 28 -> 19
Other:
- note removed: "1V1 Reg"
- note removed: "1V8 Reg"
- note removed: "2V5 Reg"
- note removed: "3V3 Reg"
Changed lines of the file:
@@
 Text GLabel 2600 7050 0    50   BiDi ~ 0
 IO17
-Text GLabel 2600 7150 0    50   BiDi ~ 0
-IO18
 Text GLabel 2600 7250 0    50   BiDi ~ 0
 IO19
@@
 Text GLabel 3900 6750 0    50   BiDi ~ 0
 IO26
-Text GLabel 3900 6850 0    50   BiDi ~ 0
+Text GLabel 3900 6950 0    50   BiDi ~ 0
 IO28
-Text GLabel 3900 6950 0    50   BiDi ~ 0
+Text GLabel 3900 7050 0    50   BiDi ~ 0
 IO29
-Text GLabel 3900 7050 0    50   BiDi ~ 0
+Text GLabel 3900 7150 0    50   BiDi ~ 0
 IO30
-Text GLabel 3900 7150 0    50   BiDi ~ 0
+Text GLabel 3900 7250 0    50   BiDi ~ 0
 IO31
-Text GLabel 3900 7250 0    50   BiDi ~ 0
+Text GLabel 3900 7350 0    50   BiDi ~ 0
 IO32
-Text GLabel 3900 7350 0    50   BiDi ~ 0
-IO33
 Text GLabel 5300 6650 0    50   BiDi ~ 0
 IO34
@@
 	0    1    1    0
 $EndComp
-$Comp
-L LFE5UM-25F-7MG285C:LFE5UM-25F-7MG285C U?
-U 10 1 5F040ECD
-P 3900 1850
-AR Path="/5BC231CE/5F040ECD" Ref="U?"  Part="10"
-AR Path="/5BC231CB/5F040ECD" Ref="U?"  Part="10"
-AR Path="/5F040ECD" Ref="U1"  Part="10"
-F 0 "U1" H 3850 2400 50  0000 C CNN
-F 1 "LFE5UM-25F-7MG285C" H 3800 2250 50  0000 C CNN
-F 2 "footprints:BGA285N50P18X18_1000X1000X130N" H 3900 1850 50  0001 L BNN
-F 3 "1.3" H 3900 1850 50  0001 L BNN
-F 4 "18.0" H 3900 1850 50  0001 L BNN "Field4"
-F 5 "18.0" H 3900 1850 50  0001 L BNN "Field5"
-F 6 "1.0" H 3900 1850 50  0001 L BNN "Field6"
-F 7 "" H 3900 1850 50  0001 L BNN "Field7"
-F 8 "1.3" H 3900 1850 50  0001 L BNN "Field8"
-F 9 "" H 3900 1850 50  0001 L BNN "Field9"
-F 10 "" H 3900 1850 50  0001 L BNN "Field10"
-F 11 "10.0" H 3900 1850 50  0001 L BNN "Field11"
-F 12 "" H 3900 1850 50  0001 L BNN "Field12"
-F 13 "" H 3900 1850 50  0001 L BNN "Field13"
-F 14 "" H 3900 1850 50  0001 L BNN "Field14"
-F 15 "" H 3900 1850 50  0001 L BNN "Field15"
-F 16 "Lattice Semiconductor" H 3900 1850 50  0001 L BNN "Field16"
-F 17 "IPC 7351B" H 3900 1850 50  0001 L BNN "Field17"
-F 18 "10.0" H 3900 1850 50  0001 L BNN "Field18"
-F 19 "False" H 3900 1850 50  0001 L BNN "Field19"
-F 20 "" H 3900 1850 50  0001 L BNN "Field20"
-F 21 "1.3" H 3900 1850 50  0001 L BNN "Field21"
-F 22 "" H 3900 1850 50  0001 L BNN "Field22"
-F 23 "10.0" H 3900 1850 50  0001 L BNN "Field23"
-F 24 "10.0" H 3900 1850 50  0001 L BNN "Field24"
-F 25 "10.0" H 3900 1850 50  0001 L BNN "Field25"
-F 26 "" H 3900 1850 50  0001 L BNN "Field26"
-F 27 "0.5" H 3900 1850 50  0001 L BNN "Field27"
-F 28 "0.3" H 3900 1850 50  0001 L BNN "Field28"
-F 29 "True" H 3900 1850 50  0001 L BNN "Field29"
-F 30 "" H 3900 1850 50  0001 L BNN "Field30"
-F 31 "" H 3900 1850 50  0001 L BNN "Field31"
-F 32 "0.5" H 3900 1850 50  0001 L BNN "Field32"
-F 33 "" H 3900 1850 50  0001 L BNN "Field33"
-F 34 "" H 3900 1850 50  0001 L BNN "Field34"
-F 35 "10.0" H 3900 1850 50  0001 L BNN "Field35"
-F 36 "" H 3900 1850 50  0001 L BNN "Field36"
-	10   3900 1850
-	1    0    0    -1
-$EndComp
-$Comp
-L power:+1V1 #PWR?
-U 1 1 5F040EE1
-P 4700 1300
-AR Path="/5BC231CB/5F040EE1" Ref="#PWR?"  Part="1"
-AR Path="/5F040EE1" Ref="#PWR0101"  Part="1"
-F 0 "#PWR0101" H 4700 1150 50  0001 C CNN
-F 1 "+1V1" V 4715 1428 50  0000 L CNN
-F 2 "" H 4700 1300 50  0001 C CNN
-F 3 "" H 4700 1300 50  0001 C CNN
-	1    4700 1300
-	0    1    1    0
-$EndComp
-$Comp
-L power:+2V5 #PWR?
-U 1 1 5F040EE7
-P 4700 1600
-AR Path="/5BC231CB/5F040EE7" Ref="#PWR?"  Part="1"
-AR Path="/5F040EE7" Ref="#PWR0102"  Part="1"
-F 0 "#PWR0102" H 4700 1450 50  0001 C CNN
-F 1 "+2V5" V 4715 1728 50  0000 L CNN
-F 2 "" H 4700 1600 50  0001 C CNN
-F 3 "" H 4700 1600 50  0001 C CNN
-	1    4700 1600
-	0    1    1    0
-$EndComp
-$Comp
-L power:+1V1 #PWR?
-U 1 1 5F040EED
-P 4700 1850
-AR Path="/5BC231CB/5F040EED" Ref="#PWR?"  Part="1"
-AR Path="/5F040EED" Ref="#PWR0103"  Part="1"
-F 0 "#PWR0103" H 4700 1700 50  0001 C CNN
-F 1 "+1V1" V 4715 1978 50  0000 L CNN
-F 2 "" H 4700 1850 50  0001 C CNN
-F 3 "" H 4700 1850 50  0001 C CNN
-	1    4700 1850
-	0    1    1    0
-$EndComp
-Wire Wire Line
-	4700 1850 4700 1950
-Connection ~ 4700 1850
-Connection ~ 4700 1950
-Wire Wire Line
-	4700 1950 4700 2050
-Connection ~ 4700 2050
-Wire Wire Line
-	4700 2050 4700 2150
-$Comp
-L power:GND #PWR?
-U 1 1 5F040EF9
-P 4700 2450
-AR Path="/5BC231CB/5F040EF9" Ref="#PWR?"  Part="1"
-AR Path="/5F040EF9" Ref="#PWR0104"  Part="1"
-F 0 "#PWR0104" H 4700 2200 50  0001 C CNN
-F 1 "GND" V 4705 2322 50  0000 R CNN
-F 2 "" H 4700 2450 50  0001 C CNN
-F 3 "" H 4700 2450 50  0001 C CNN
-	1    4700 2450
-	0    -1   -1   0
-$EndComp
-Wire Wire Line
-	4700 1250 4700 1300
-Connection ~ 4700 1300
-Wire Wire Line
-	4700 1300 4700 1350
-Wire Wire Line
-	4700 1550 4700 1600
-Connection ~ 4700 1600
-Wire Wire Line
-	4700 1600 4700 1650
-Text Notes 5600 6200 0    50   ~ 0
-1V1 Reg
-Text Notes 5600 6300 0    50   ~ 0
-1V8 Reg
-Text Notes 5600 6400 0    50   ~ 0
-2V5 Reg
-Text Notes 5600 6500 0    50   ~ 0
-3V3 Reg
 Wire Wire Line
 	7550 1800 8550 1800
@@
 Wire Wire Line
 	7550 3200 8550 3200
-Wire Wire Line
-	8550 3100 7550 3100
-Wire Wire Line
-	7550 3000 8550 3000
 $Sheet
 S 5700 1250 1850 2650
@@
 F9 "FLASH_MOSI" B R 7550 2000 50
 F10 "FLASH_SCK" B R 7550 1900 50
-F11 "DONE" B R 7550 3000 50
-F12 "INITN" B R 7550 3100 50
-F13 "PROGRAMN" B R 7550 3200 50
-F14 "FLASH_HOLD" I R 7550 1800 50
+F11 "PROGRAMN" B R 7550 3200 50
+F12 "FLASH_HOLD" I R 7550 1800 50
 $EndSheet
 $Sheet
@@
 F6 "SDIO1_DAT3" B L 8550 2800 50
 F7 "SDIO1_DAT0" B L 8550 2500 50
-F8 "FPGA_DONE" B L 8550 3000 50
-F9 "FPGA_PROGRAMN" B L 8550 3200 50
-F10 "INITN" B L 8550 3100 50
-F11 "FLASH_MISO" B L 8550 2100 50
-F12 "FLASH_MOSI" B L 8550 2000 50
-F13 "FLASH_CLK" B L 8550 1900 50
-F14 "FLASH_HOLD" B L 8550 1800 50
+F8 "FPGA_PROGRAMN" B L 8550 3200 50
+F9 "FLASH_MISO" B L 8550 2100 50
+F10 "FLASH_MOSI" B L 8550 2000 50
+F11 "FLASH_CLK" B L 8550 1900 50
+F12 "FLASH_HOLD" B L 8550 1800 50
 $EndSheet
 Wire Wire Line
@@
 	0    1    1    0
 $EndComp
-Text GLabel 5300 6450 0    50   Input ~ 0
-EN
 $Comp
 L Mechanical:MountingHole_Pad H3
@@
 	1    0    0    -1
 $EndComp
+Text GLabel 5300 6550 0    50   BiDi ~ 0
+IO33
+Text GLabel 3900 6850 0    50   BiDi ~ 0
+IO27
+Text GLabel 2600 7150 0    50   BiDi ~ 0
+IO18
+Text GLabel 5300 6450 0    50   Output ~ 0
+EN
 $EndSCHEMATC

Commit message: FPGA_ESP32 : progress on power and replaced sdio by qspi
Connections:
- net labels added: SPI_CLK, SPI_HD, SPI_MISO, SPI_MOSI, SPI_WP
- net labels removed: IO38, IO39, IO40, IO41
- wire segments 19 -> 12
Changed lines of the file:
@@
 	0    -1   1    0
 $EndComp
-Text GLabel 1300 6550 0    50   BiDi ~ 0
-IO0
-Text GLabel 1300 6650 0    50   BiDi ~ 0
-IO1
-Text GLabel 1300 6750 0    50   BiDi ~ 0
-IO2
-Text GLabel 1300 6850 0    50   BiDi ~ 0
-IO3
-Text GLabel 1300 6950 0    50   BiDi ~ 0
-IO4
-Text GLabel 1300 7050 0    50   BiDi ~ 0
-IO5
-Text GLabel 1300 7150 0    50   BiDi ~ 0
-IO6
-Text GLabel 1300 7250 0    50   BiDi ~ 0
-IO7
-Text GLabel 1300 7350 0    50   BiDi ~ 0
-IO8
-Text GLabel 2600 6250 0    50   BiDi ~ 0
-IO9
-Text GLabel 2600 6350 0    50   BiDi ~ 0
-IO10
-Text GLabel 2600 6450 0    50   BiDi ~ 0
-IO11
-Text GLabel 2600 6550 0    50   BiDi ~ 0
-IO12
-Text GLabel 2600 6650 0    50   BiDi ~ 0
-IO13
-Text GLabel 2600 6750 0    50   BiDi ~ 0
-IO14
-Text GLabel 2600 6850 0    50   BiDi ~ 0
-IO15
-Text GLabel 2600 6950 0    50   BiDi ~ 0
-IO16
-Text GLabel 2600 7050 0    50   BiDi ~ 0
-IO17
-Text GLabel 2600 7250 0    50   BiDi ~ 0
-IO19
-Text GLabel 2600 7350 0    50   BiDi ~ 0
-IO20
-Text GLabel 3900 6250 0    50   BiDi ~ 0
-IO21
 Text GLabel 2600 6050 0    50   Input ~ 0
 VIO
-Text GLabel 3900 6350 0    50   BiDi ~ 0
-IO22
-Text GLabel 3900 6450 0    50   BiDi ~ 0
-IO23
-Text GLabel 3900 6550 0    50   BiDi ~ 0
-IO24
-Text GLabel 3900 6650 0    50   BiDi ~ 0
-IO25
-Text GLabel 3900 6750 0    50   BiDi ~ 0
-IO26
-Text GLabel 3900 6950 0    50   BiDi ~ 0
-IO28
-Text GLabel 3900 7050 0    50   BiDi ~ 0
-IO29
-Text GLabel 3900 7150 0    50   BiDi ~ 0
-IO30
-Text GLabel 3900 7250 0    50   BiDi ~ 0
-IO31
-Text GLabel 3900 7350 0    50   BiDi ~ 0
-IO32
-Text GLabel 5300 6650 0    50   BiDi ~ 0
-IO34
-Text GLabel 5300 6750 0    50   BiDi ~ 0
-IO35
-Text GLabel 5300 6850 0    50   BiDi ~ 0
-IO36
-Text GLabel 5300 6950 0    50   BiDi ~ 0
-IO37
-Text GLabel 5300 7050 0    50   BiDi ~ 0
-IO38
-Text GLabel 5300 7150 0    50   BiDi ~ 0
-IO39
-Text GLabel 5300 7250 0    50   BiDi ~ 0
-IO40
 $Comp
 L power:GND #PWR0106
@@
 	7550 1800 8550 1800
 Wire Wire Line
-	7550 2100 8550 2100
-Wire Wire Line
-	8550 2000 7550 2000
-Wire Wire Line
-	7550 1900 8550 1900
-Wire Wire Line
 	7550 3200 8550 3200
 $Sheet
@@
 F0 "FPGA" 50
 F1 "io.sch" 50
-F2 "SDIO1_CLK" B R 7550 2300 50
-F3 "SDIO1_CMD" B R 7550 2400 50
-F4 "SDIO1_DAT1" B R 7550 2600 50
-F5 "SDIO1_DAT2" B R 7550 2700 50
-F6 "SDIO1_DAT3" B R 7550 2800 50
-F7 "SDIO1_DAT0" B R 7550 2500 50
-F8 "FLASH_MISO" B R 7550 2100 50
-F9 "FLASH_MOSI" B R 7550 2000 50
-F10 "FLASH_SCK" B R 7550 1900 50
-F11 "PROGRAMN" B R 7550 3200 50
-F12 "FLASH_HOLD" I R 7550 1800 50
+F2 "PROGRAMN" B R 7550 3200 50
+F3 "FPGA_MISO" B R 7550 2100 50
+F4 "FPGA_MOSI" B R 7550 2000 50
+F5 "FPGA_SCK" B R 7550 1900 50
+F6 "FPGA_CS" B R 7550 1800 50
+F7 "FPGA_HOLDN" B R 7550 3000 50
+F8 "DONE" B R 7550 3100 50
+F9 "FPGA_IO2" B R 7550 1700 50
+F10 "FPGA_IO3" B R 7550 1600 50
 $EndSheet
 $Sheet
@@
 F0 "WIFI, BT, RT" 50
 F1 "esp32.sch" 50
-F2 "SDIO1_CLK" B L 8550 2300 50
-F3 "SDIO1_CMD" B L 8550 2400 50
-F4 "SDIO1_DAT1" B L 8550 2600 50
-F5 "SDIO1_DAT2" B L 8550 2700 50
-F6 "SDIO1_DAT3" B L 8550 2800 50
-F7 "SDIO1_DAT0" B L 8550 2500 50
-F8 "FPGA_PROGRAMN" B L 8550 3200 50
-F9 "FLASH_MISO" B L 8550 2100 50
-F10 "FLASH_MOSI" B L 8550 2000 50
-F11 "FLASH_CLK" B L 8550 1900 50
-F12 "FLASH_HOLD" B L 8550 1800 50
+F2 "FPGA_PROGRAMN" B L 8550 3200 50
+F3 "SPI_MISO" B L 8550 2100 50
+F4 "SPI_CLK" B L 8550 1900 50
+F5 "SPI_MOSI" B L 8550 2000 50
+F6 "FPGA_CS" B L 8550 1800 50
+F7 "SPI_WP" B L 8550 1700 50
+F8 "SPI_HD" B L 8550 1600 50
+F9 "FPGA_DONE" B L 8550 3100 50
+F10 "FPGA_HOLD" B L 8550 3000 50
 $EndSheet
-Wire Wire Line
-	8550 2800 7550 2800
-Wire Wire Line
-	7550 2700 8550 2700
-Wire Wire Line
-	8550 2600 7550 2600
-Wire Wire Line
-	7550 2500 8550 2500
-Wire Wire Line
-	8550 2400 7550 2400
-Wire Wire Line
-	7550 2300 8550 2300
 $Comp
 L power:GND #PWR0112
@@
 	0    1    1    0
 $EndComp
-Text GLabel 5300 7350 0    50   BiDi ~ 0
-IO41
 $Comp
 L power:GND #PWR0111
@@
 	1    0    0    -1
 $EndComp
-Text GLabel 5300 6550 0    50   BiDi ~ 0
-IO33
+Text GLabel 5300 6450 0    50   Output ~ 0
+EN
+Wire Wire Line
+	8550 3100 7550 3100
+Wire Wire Line
+	8550 3000 7550 3000
+Text Label 8550 1600 2    50   ~ 0
+SPI_HD
+Text Label 8550 1700 2    50   ~ 0
+SPI_WP
+Text Label 8550 1900 2    50   ~ 0
+SPI_CLK
+Text Label 8550 2000 2    50   ~ 0
+SPI_MOSI
+Text Label 8550 2100 2    50   ~ 0
+SPI_MISO
+Text Label 7550 1900 0    50   ~ 0
+SPI_CLK
+Text Label 7550 2000 0    50   ~ 0
+SPI_MOSI
+Text Label 7550 2100 0    50   ~ 0
+SPI_MISO
+Text Label 7550 1600 0    50   ~ 0
+SPI_HD
+Text Label 7550 1700 0    50   ~ 0
+SPI_WP
+Text Label 5300 6750 2    50   ~ 0
+SPI_CLK
+Text Label 5300 6850 2    50   ~ 0
+SPI_MOSI
+Text Label 5300 6950 2    50   ~ 0
+SPI_MISO
+Text Label 5300 6550 2    50   ~ 0
+SPI_HD
+Text Label 5300 6650 2    50   ~ 0
+SPI_WP
+Text GLabel 1300 6550 0    50   BiDi ~ 0
+IO0
+Text GLabel 1300 6650 0    50   BiDi ~ 0
+IO1
+Text GLabel 1300 6750 0    50   BiDi ~ 0
+IO2
+Text GLabel 1300 6850 0    50   BiDi ~ 0
+IO3
+Text GLabel 1300 6950 0    50   BiDi ~ 0
+IO4
+Text GLabel 1300 7050 0    50   BiDi ~ 0
+IO5
+Text GLabel 1300 7150 0    50   BiDi ~ 0
+IO6
+Text GLabel 1300 7250 0    50   BiDi ~ 0
+IO7
+Text GLabel 1300 7350 0    50   BiDi ~ 0
+IO8
+Text GLabel 2600 6250 0    50   BiDi ~ 0
+IO9
+Text GLabel 2600 6350 0    50   BiDi ~ 0
+IO10
+Text GLabel 2600 6450 0    50   BiDi ~ 0
+IO11
+Text GLabel 2600 6550 0    50   BiDi ~ 0
+IO12
+Text GLabel 2600 6650 0    50   BiDi ~ 0
+IO13
+Text GLabel 2600 6850 0    50   BiDi ~ 0
+IO15
+Text GLabel 2600 6950 0    50   BiDi ~ 0
+IO16
+Text GLabel 2600 7050 0    50   BiDi ~ 0
+IO17
+Text GLabel 2600 7150 0    50   BiDi ~ 0
+IO18
+Text GLabel 2600 7250 0    50   BiDi ~ 0
+IO19
+Text GLabel 2600 7350 0    50   BiDi ~ 0
+IO20
+Text GLabel 3900 6250 0    50   BiDi ~ 0
+IO21
+Text GLabel 3900 6750 0    50   BiDi ~ 0
+IO26
 Text GLabel 3900 6850 0    50   BiDi ~ 0
 IO27
-Text GLabel 2600 7150 0    50   BiDi ~ 0
-IO18
-Text GLabel 5300 6450 0    50   Output ~ 0
-EN
+Text GLabel 3900 6450 0    50   BiDi ~ 0
+IO23
+Text GLabel 3900 6350 0    50   BiDi ~ 0
+IO22
+Text GLabel 3900 6550 0    50   BiDi ~ 0
+IO24
+Text GLabel 2600 6750 0    50   BiDi ~ 0
+IO14
+Text GLabel 3900 6650 0    50   BiDi ~ 0
+IO25
+Text GLabel 3900 7250 0    50   BiDi ~ 0
+IO31
+Text GLabel 3900 7350 0    50   BiDi ~ 0
+IO32
+Text GLabel 5300 7050 0    50   BiDi ~ 0
+IO33
+Text GLabel 5300 7150 0    50   BiDi ~ 0
+IO34
+Text GLabel 5300 7250 0    50   BiDi ~ 0
+IO35
+Text GLabel 3900 6950 0    50   BiDi ~ 0
+IO28
+Text GLabel 3900 7050 0    50   BiDi ~ 0
+IO29
+Text GLabel 3900 7150 0    50   BiDi ~ 0
+IO30
+Text GLabel 5300 7350 0    50   BiDi ~ 0
+IO36
 $EndSCHEMATC
