File: FPGA_ESP32/io.sch (KiCad schematic (older format))
At the start: 21 parts

Commit message: FPGA_ESP32 : add header + esp32 with SDIO
Parts:
- removed C?: 100nF, symbol Device:C
- removed U?: LY68L6400SLIT, symbol Lyontek_psram:LY68L6400SLIT
- added C7: 10nF, Capacitor_SMD:C_0402_1005Metric, symbol Device:C
- added C? (x5): 100nF, symbol Device:C
- added J2: CAM, fpc_cam24:FPC_24_CAM, symbol Connector:Conn_01x24_Female
- added R1: 1K, Resistor_SMD:R_0201_0603Metric, symbol Device:R
- added R2, R3, R4, R5, R? (x3): 4K7, symbol Device:R
- added U3: BMP280, Package_LGA:Bosch_LGA-8_2x2.5mm_P0.65mm_ClockwisePinNumbering, symbol Sensor_Pressure:BMP280
- added U5: ICM-20948, Sensor_Motion:InvenSense_QFN-24_3x3mm_P0.4mm, symbol Sensor_Motion:ICM-20948
- C1, C2, C3, C4, C5: renamed from C?; footprint (none) -> Capacitor_SMD:C_0402_1005Metric
- U1: renamed from U?; footprint BGA285N50P18X18_1000X1000X130N -> footprints:BGA285N50P18X18_1000X1000X130N
- U4, U6, U7, U8, U9: renamed from U?; footprint (none) -> Package_SO:SSOP-8_3.9x5.05mm_P1.27mm
Connections:
- net labels added: +1V8, +2V8, 1V8_I2C_SCL, 1V8_I2C_SDA, ADCREF, ADCREFOUT, DONE, FLASH_MISO, FLASH_MOSI, FLASH_SCK, ICM_INT, INITN, IO0, IO1, IO10, IO11, IO12, IO19, IO2, IO20, IO21, IO22, IO23, IO24, IO25, IO26, IO27, IO28, IO29, IO3, IO30, IO31, IO32, IO4, IO5, IO6, IO7, IO8, IO9, PROGRAMN, TCK, TDI, TDO, TMS
- net labels removed: CAM_AVDD, CAM_DOVDD, CSI_Y0, CSI_Y1, RAM5_CE, RAM5_SCLK, RAM5_SIO0, RAM5_SIO1, RAM5_SIO3, RAM5_SIO4, STROBE
- wire segments 1 -> 25
- no-connect marks 12 -> 18
Other:
- note added: "5 * PSRAM QSPI LY68L6400\n4 for Image Processing\n1 for SoftCore"
- note added: "BMP280 @0x76"
- note added: "ICM-20948 @0x68"
- note added: "OV5640 @0x78"
- moved on the sheet: C1, C2, C3, C4, C5, U1E, U1F, U4, U6, U7, U8, U9

Commit message: FPGA_ESP32 : add 2 psram ic, rf switch
Parts:
- removed C2, C3, C4, C5: 100nF, Capacitor_SMD:C_0402_1005Metric, symbol Device:C
- removed C? (x5): 100nF, symbol Device:C
- removed U3: BMP280, Package_LGA:Bosch_LGA-8_2x2.5mm_P0.65mm_ClockwisePinNumbering, symbol Sensor_Pressure:BMP280
- removed U4, U6, U7, U8, U9: LY68L6400SLIT, Package_SO:SSOP-8_3.9x5.05mm_P1.27mm, symbol Lyontek_psram:LY68L6400SLIT
- removed U5: ICM-20948, Sensor_Motion:InvenSense_QFN-24_3x3mm_P0.4mm, symbol Sensor_Motion:ICM-20948
- added R15: R, Resistor_SMD:R_0201_0603Metric, symbol Device:R
- added U4, U6: W956D6KBKX, footprints:BGA-49_7x7_4.0x4.0mm, symbol ob:W956D6KBKX
- R12, R13, R14: renamed from R?; footprint (none) -> Resistor_SMD:R_0201_0603Metric
- R2, R3, R4, R5: footprint (none) -> Resistor_SMD:R_0201_0603Metric
Connections:
- net labels added: IO36, IO37, RAM0_A16, RAM0_A17, RAM0_A18, RAM0_A19, RAM0_A20, RAM0_A21, RAM0_ADQ0, RAM0_ADQ1, RAM0_ADQ10, RAM0_ADQ11, RAM0_ADQ12, RAM0_ADQ13, RAM0_ADQ14, RAM0_ADQ15, RAM0_ADQ2, RAM0_ADQ3, RAM0_ADQ4, RAM0_ADQ5, RAM0_ADQ6, RAM0_ADQ7, RAM0_ADQ8, RAM0_ADQ9, RAM1_A16, RAM1_A17, RAM1_A18, RAM1_A19, RAM1_A20, RAM1_A21, RAM1_ADQ0, RAM1_ADQ1, RAM1_ADQ10, RAM1_ADQ11, RAM1_ADQ12, RAM1_ADQ13, RAM1_ADQ14, RAM1_ADQ15, RAM1_ADQ2, RAM1_ADQ3, RAM1_ADQ4, RAM1_ADQ5, RAM1_ADQ6, RAM1_ADQ7, RAM1_ADQ8, RAM1_ADQ9, RAM2_ADQ10, RAM2_ADQ11, RAM2_ADQ12, RAM2_ADQ13, RAM2_ADQ8, RAM2_ADQ9, RAM_WAIT
- net labels removed: 1V8_I2C_SCL, 1V8_I2C_SDA, ICM_INT, RAM0_CE, RAM0_SCLK, RAM0_SIO0, RAM0_SIO1, RAM0_SIO3, RAM0_SIO4, RAM1_CE, RAM1_SCLK, RAM1_SIO0, RAM1_SIO1, RAM1_SIO3, RAM1_SIO4, RAM2_CE, RAM2_SCLK, RAM2_SIO0, RAM2_SIO1, RAM2_SIO3, RAM2_SIO4, RAM3_CE, RAM3_SCLK, RAM3_SIO0, RAM3_SIO1, RAM3_SIO3, RAM3_SIO4, RAM4_CE, RAM4_SCLK, RAM4_SIO0, RAM4_SIO1, RAM4_SIO3, RAM4_SIO4, TCK, TDI, TDO, TMS
- wire segments 25 -> 11
- no-connect marks 18 -> 14
Other:
- note added: "1V8 I2C SCL"
- note added: "1V8 I2C SDA"
- note removed: "5 * PSRAM QSPI LY68L6400\n4 for Image Processing\n1 for SoftCore"
- note removed: "BMP280 @0x76"
- note removed: "ICM-20948 @0x68"
- moved on the sheet: C1

Commit message: FPGA_ESP32 : add camera, change header position
Parts:
- added D1: LED_RGBC, LED_SMD:LED_Cree-PLCC4_2x2mm_CW, symbol Device:LED_RGBC
Connections:
- net labels added: FLASH_HOLD, IO15, IO16, IO34, IO38, IO39
- net labels removed: RAM2_ADQ10, RAM2_ADQ11, RAM2_ADQ12, RAM2_ADQ13, RAM2_ADQ8, RAM2_ADQ9
Other:
- moved on the sheet: U1A, U1B

Commit message: FPGA_ESP32 : lot of fix + modification
Replace digital camera by analog camera decoder
Fix PSRAM io domain 3.3V -> 1.8V
Start reducing capacitor number
Add remaining psram pin
Sheet resize
Parts:
- removed D1: LED_RGBC, LED_SMD:LED_Cree-PLCC4_2x2mm_CW, symbol Device:LED_RGBC
- removed J2: CAM, fpc_cam24:FPC_24_CAM, symbol Connector:Conn_01x24_Female
- removed R1: 1K, Resistor_SMD:R_0201_0603Metric, symbol Device:R
- removed R15: R, Resistor_SMD:R_0201_0603Metric, symbol Device:R
- removed R2, R3, R4: 4K7, Resistor_SMD:R_0201_0603Metric, symbol Device:R
- removed unit 5 of U1
- added C14: 10uF, Capacitor_SMD:C_0402_1005Metric, symbol Device:C
- added C15, C16: 0.1uF, Capacitor_SMD:C_0402_1005Metric, symbol Device:C
- added C17: C, Capacitor_SMD:C_0402_1005Metric, symbol Device:C
- added U5: TW9900, footprints:QFN-32_EP_4x4_Pitch0.4mm, symbol ob:TW9900
- added Y1: Crystal_GND23, symbol Device:Crystal_GND23
- C7: value 10nF -> C
- R12, R13: value 4K7 -> 4.7K
- R5: value 4K7 -> 1M
Connections:
- net labels added: AVIN1, AVIN2, HSYNC, IO41, MPOUT, RAM0_ADV, RAM0_CE, RAM0_CLK, RAM0_CRE, RAM0_LB, RAM0_OE, RAM0_UB, RAM0_WAIT, RAM0_WE, RAM1_ADV, RAM1_CE, RAM1_CLK, RAM1_CRE, RAM1_LB, RAM1_OE, RAM1_UB, RAM1_WAIT, RAM1_WE, TW_I2C_DAT, TW_I2C_SCK, TW_INT, TW_PWRDN, VIN_CLK, VIN_D0, VIN_D1, VIN_D2, VIN_D3, VIN_D4, VIN_D5, VIN_D6, VIN_D7, VSYNC, nRESET
- net labels removed: +2V8, ADCREF, ADCREFOUT, CSI_HSYNC, CSI_I2C_SCL, CSI_I2C_SDA, CSI_MCLK, CSI_PCLK, CSI_PWDN, CSI_VSYNC, CSI_Y2, CSI_Y3, CSI_Y4, CSI_Y5, CSI_Y6, CSI_Y7, CSI_Y8, CSI_Y9, IO27, IO31, IO32, IO36, IO37, RAM_WAIT, ~CSI_RST
- wire segments 11 -> 48
- no-connect marks 14 -> 10
Other:
- note removed: "1V8 I2C SCL"
- note removed: "1V8 I2C SDA"
- note removed: "OV5640 @0x78"
- moved on the sheet: C1, R14, U1A, U1B, U1C, U1F, U1G, U1H, U1I

Commit message: FPGA_ESP32 : esp32 enable circuit, flash done, more doc, TODO power !
Parts:
- removed C1: 100nF, Capacitor_SMD:C_0402_1005Metric, symbol Device:C
- added C? (x2): 0.1uF, Capacitor_SMD:C_0402_1005Metric, symbol Device:C
- added C? (x2): 10uF, Capacitor_SMD:C_0402_1005Metric, symbol Device:C
- added R?: 4.7K, symbol Device:R
- added unit 10 of U1
- added U?: TLV71211_SOT23-5, Package_TO_SOT_SMD:SOT-23-5, symbol Regulator_Linear:TLV71211_SOT23-5
- added U?: SPX3819M5-L-1-8, Package_TO_SOT_SMD:SOT-23-5, symbol Regulator_Linear:SPX3819M5-L-1-8
- added U?: LD1117S25TR_SOT223, Package_TO_SOT_SMD:SOT-223-3_TabPin2, symbol Regulator_Linear:LD1117S25TR_SOT223
Connections:
- net labels added: +1V1, +2V5, IO33
- net labels removed: DONE, FLASH_HOLD, INITN
- wire segments 48 -> 77
- no-connect marks 10 -> 11
Other:
- note added: "1V1 Reg"
- note added: "1V8 Reg"
- note added: "2V5 Reg"
- moved on the sheet: R14

Commit message: FPGA_ESP32 : progress on power and replaced sdio by qspi
Parts:
- removed U?: LD1117S25TR_SOT223, Package_TO_SOT_SMD:SOT-223-3_TabPin2, symbol Regulator_Linear:LD1117S25TR_SOT223
- added U9: SPX3819M5-L-2-5, Package_TO_SOT_SMD:SOT-23-5, symbol Regulator_Linear:SPX3819M5-L-2-5
- R7: renamed from R?; footprint (none) -> Resistor_SMD:R_0201_0603Metric
- Y1: footprint (none) -> Crystal:Crystal_SMD_2520-4Pin_2.5x2.0mm
- gave numbers to parts that had none: 6
Connections:
- net labels added: DONE, FPGA_CS, FPGA_HOLDN, FPGA_IO2, FPGA_IO3, FPGA_MISO, FPGA_MOSI, FPGA_SCK, IO13, IO14, IO17, IO18, IO27
- net labels removed: FLASH_MISO, FLASH_MOSI, FLASH_SCK, IO28, IO29, IO30, IO33, IO34, IO38, IO39, IO41, SDIO1_CLK, SDIO1_CMD, SDIO1_DAT0, SDIO1_DAT1, SDIO1_DAT2, SDIO1_DAT3
- wire segments 77 -> 76
- no-connect marks 11 -> 15

Commit message: FPGA_ESP32 : power done, antenna matching done, todo crystal and capacitor purge
Parts:
- removed U3: TLV71211_SOT23-5, Package_TO_SOT_SMD:SOT-23-5, symbol Regulator_Linear:TLV71211_SOT23-5
- removed U8: SPX3819M5-L-1-8, Package_TO_SOT_SMD:SOT-23-5, symbol Regulator_Linear:SPX3819M5-L-1-8
- removed U9: SPX3819M5-L-2-5, Package_TO_SOT_SMD:SOT-23-5, symbol Regulator_Linear:SPX3819M5-L-2-5
- added C19, C20, C21: 1uF, Capacitor_SMD:C_0402_1005Metric, symbol Device:C
- added U3: LP5910, footprints:BGA-4_2x2_0.74x0.74mm, symbol ob:LP5910
- added U8: ADP222ACPZ-1825-R7, footprints:SON50P200X200X60-9N, symbol ob:ADP222ACPZ-1825-R7
Connections:
- wire segments 76 -> 83
Changed lines of the file:
@@
 Wire Wire Line
 	4550 1450 4550 1500
-Text Notes 6500 800  0    50   ~ 0
+Text Notes 6300 800  0    50   ~ 0
 1V1 Reg
-Text Notes 7800 850  0    50   ~ 0
-1V8 Reg
-Text Notes 9150 850  0    50   ~ 0
-2V5 Reg
-$Comp
-L Regulator_Linear:TLV71211_SOT23-5 U3
-U 1 1 5F9A1612
-P 6700 1250
-F 0 "U3" H 6700 1592 50  0000 C CNN
-F 1 "TLV71211_SOT23-5" H 6700 1501 50  0000 C CNN
-F 2 "Package_TO_SOT_SMD:SOT-23-5" H 6700 1575 50  0001 C CIN
-F 3 "http://www.ti.com/lit/ds/symlink/tlv712.pdf" H 6700 1300 50  0001 C CNN
-	1    6700 1250
-	1    0    0    -1
-$EndComp
-$Comp
-L Regulator_Linear:SPX3819M5-L-1-8 U8
-U 1 1 5F9A7D86
-P 8000 1250
-F 0 "U8" H 8000 1592 50  0000 C CNN
-F 1 "SPX3819M5-L-1-8" H 8000 1501 50  0000 C CNN
-F 2 "Package_TO_SOT_SMD:SOT-23-5" H 8000 1575 50  0001 C CNN
-F 3 "https://www.exar.com/content/document.ashx?id=22106&languageid=1033&type=Datasheet&partnumber=SPX3819&filename=SPX3819.pdf&part=SPX3819" H 8000 1250 50  0001 C CNN
-	1    8000 1250
-	1    0    0    -1
-$EndComp
-Text GLabel 6150 1200 0    50   Input ~ 0
+Text GLabel 5950 1400 0    50   Input ~ 0
 VIO
 Text HLabel 8650 4800 2    50   BiDi ~ 0
@@
 NoConn ~ 2550 4300
 $Comp
-L Regulator_Linear:SPX3819M5-L-2-5 U9
-U 1 1 5FACFC03
-P 9350 1250
-F 0 "U9" H 9350 1592 50  0000 C CNN
-F 1 "SPX3819M5-L-2-5" H 9350 1501 50  0000 C CNN
-F 2 "Package_TO_SOT_SMD:SOT-23-5" H 9350 1575 50  0001 C CNN
-F 3 "https://www.exar.com/content/document.ashx?id=22106&languageid=1033&type=Datasheet&partnumber=SPX3819&filename=SPX3819.pdf&part=SPX3819" H 9350 1250 50  0001 C CNN
-	1    9350 1250
-	1    0    0    -1
-$EndComp
+L power:+2V5 #PWR?
+U 1 1 5F0E8E67
+P 8600 1450
+AR Path="/5BC231CB/5F0E8E67" Ref="#PWR?"  Part="1"
+AR Path="/5F0E8E67" Ref="#PWR?"  Part="1"
+AR Path="/5BC231CE/5F0E8E67" Ref="#PWR0151"  Part="1"
+F 0 "#PWR0151" H 8600 1300 50  0001 C CNN
+F 1 "+2V5" V 8615 1578 50  0000 L CNN
+F 2 "" H 8600 1450 50  0001 C CNN
+F 3 "" H 8600 1450 50  0001 C CNN
+	1    8600 1450
+	0    1    1    0
+$EndComp
+$Comp
+L power:+1V8 #PWR0152
+U 1 1 5F0EC5A4
+P 8600 1200
+AR Path="/5BC231CE/5F0EC5A4" Ref="#PWR0152"  Part="1"
+AR Path="/5BC231CB/5F0EC5A4" Ref="#PWR?"  Part="1"
+AR Path="/5F0EC5A4" Ref="#PWR?"  Part="1"
+F 0 "#PWR0152" H 8600 1050 50  0001 C CNN
+F 1 "+1V8" V 8615 1328 50  0000 L CNN
+F 2 "" H 8600 1200 50  0001 C CNN
+F 3 "" H 8600 1200 50  0001 C CNN
+	1    8600 1200
+	0    1    -1   0
+$EndComp
+$Comp
+L ob:ADP222ACPZ-1825-R7 U8
+U 1 1 5F0F4362
+P 8100 1600
+F 0 "U8" H 8100 2275 50  0000 C CNN
+F 1 "ADP222ACPZ-1825-R7" H 8100 2184 50  0000 C CNN
+F 2 "footprints:SON50P200X200X60-9N" H 8100 2200 50  0001 C CNN
+F 3 "" H 8100 2200 50  0001 C CNN
+	1    8100 1600
+	1    0    0    -1
+$EndComp
+$Comp
+L power:GND #PWR0153
+U 1 1 5F0FD413
+P 8100 1650
+F 0 "#PWR0153" H 8100 1400 50  0001 C CNN
+F 1 "GND" H 8105 1477 50  0000 C CNN
+F 2 "" H 8100 1650 50  0001 C CNN
+F 3 "" H 8100 1650 50  0001 C CNN
+	1    8100 1650
+	1    0    0    -1
+$EndComp
+$Comp
+L power:GND #PWR0154
+U 1 1 5F0FF5F1
+P 7600 1350
+F 0 "#PWR0154" H 7600 1100 50  0001 C CNN
+F 1 "GND" V 7605 1222 50  0000 R CNN
+F 2 "" H 7600 1350 50  0001 C CNN
+F 3 "" H 7600 1350 50  0001 C CNN
+	1    7600 1350
+	0    1    1    0
+$EndComp
+Text Notes 7900 800  0    50   ~ 0
+2V5 Reg
+Text Notes 7900 700  0    50   ~ 0
+1V8 Reg
+$Comp
+L Device:C C19
+U 1 1 5F121970
+P 9150 1500
+F 0 "C19" H 9265 1546 50  0000 L CNN
+F 1 "1uF" H 9265 1455 50  0000 L CNN
+F 2 "Capacitor_SMD:C_0402_1005Metric" H 9188 1350 50  0001 C CNN
+F 3 "~" H 9150 1500 50  0001 C CNN
+	1    9150 1500
+	1    0    0    -1
+$EndComp
+$Comp
+L power:GND #PWR0155
+U 1 1 5F12429C
+P 9150 1650
+F 0 "#PWR0155" H 9150 1400 50  0001 C CNN
+F 1 "GND" H 9155 1477 50  0000 C CNN
+F 2 "" H 9150 1650 50  0001 C CNN
+F 3 "" H 9150 1650 50  0001 C CNN
+	1    9150 1650
+	1    0    0    -1
+$EndComp
+Wire Wire Line
+	9150 1350 8600 1350
+Text GLabel 9150 1350 2    50   Input ~ 0
+VIO
+Wire Wire Line
+	7600 1150 7600 1250
+Text GLabel 7600 1200 0    50   Input ~ 0
+VIO
+Wire Wire Line
+	8600 1150 8600 1200
+Connection ~ 8600 1200
+Wire Wire Line
+	8600 1200 8600 1250
+$Comp
+L power:+2V5 #PWR?
+U 1 1 5F16774A
+P 7600 1450
+AR Path="/5BC231CB/5F16774A" Ref="#PWR?"  Part="1"
+AR Path="/5F16774A" Ref="#PWR?"  Part="1"
+AR Path="/5BC231CE/5F16774A" Ref="#PWR0156"  Part="1"
+F 0 "#PWR0156" H 7600 1300 50  0001 C CNN
+F 1 "+2V5" V 7615 1578 50  0000 L CNN
+F 2 "" H 7600 1450 50  0001 C CNN
+F 3 "" H 7600 1450 50  0001 C CNN
+	1    7600 1450
+	0    -1   -1   0
+$EndComp
+$Comp
+L ob:LP5910 U3
+U 1 1 5F18D5C8
+P 6450 1300
+F 0 "U3" H 6450 1465 50  0000 C CNN
+F 1 "LP5910" H 6450 1374 50  0000 C CNN
+F 2 "footprints:BGA-4_2x2_0.74x0.74mm" H 6450 1300 50  0001 C CNN
+F 3 "" H 6450 1300 50  0001 C CNN
+	1    6450 1300
+	1    0    0    -1
+$EndComp
+$Comp
+L Device:C C20
+U 1 1 5F192F78
+P 5950 1250
+F 0 "C20" H 6065 1296 50  0000 L CNN
+F 1 "1uF" H 6065 1205 50  0000 L CNN
+F 2 "Capacitor_SMD:C_0402_1005Metric" H 5988 1100 50  0001 C CNN
+F 3 "~" H 5950 1250 50  0001 C CNN
+	1    5950 1250
+	1    0    0    1
+$EndComp
+$Comp
+L power:GND #PWR0157
+U 1 1 5F192F7E
+P 5950 1100
+F 0 "#PWR0157" H 5950 850 50  0001 C CNN
+F 1 "GND" H 5955 927 50  0000 C CNN
+F 2 "" H 5950 1100 50  0001 C CNN
+F 3 "" H 5950 1100 50  0001 C CNN
+	1    5950 1100
+	1    0    0    1
+$EndComp
+$Comp
+L Device:C C21
+U 1 1 5F19B819
+P 6800 1250
+F 0 "C21" H 6915 1296 50  0000 L CNN
+F 1 "1uF" H 6915 1205 50  0000 L CNN
+F 2 "Capacitor_SMD:C_0402_1005Metric" H 6838 1100 50  0001 C CNN
+F 3 "~" H 6800 1250 50  0001 C CNN
+	1    6800 1250
+	1    0    0    1
+$EndComp
+$Comp
+L power:GND #PWR0158
+U 1 1 5F19B81F
+P 6800 1100
+F 0 "#PWR0158" H 6800 850 50  0001 C CNN
+F 1 "GND" H 6805 927 50  0000 C CNN
+F 2 "" H 6800 1100 50  0001 C CNN
+F 3 "" H 6800 1100 50  0001 C CNN
+	1    6800 1100
+	1    0    0    1
+$EndComp
+$Comp
+L power:+1V1 #PWR?
+U 1 1 5F1ADB23
+P 6800 1400
+AR Path="/5BC231CB/5F1ADB23" Ref="#PWR?"  Part="1"
+AR Path="/5F1ADB23" Ref="#PWR?"  Part="1"
+AR Path="/5BC231CE/5F1ADB23" Ref="#PWR0159"  Part="1"
+F 0 "#PWR0159" H 6800 1250 50  0001 C CNN
+F 1 "+1V1" V 6815 1528 50  0000 L CNN
+F 2 "" H 6800 1400 50  0001 C CNN
+F 3 "" H 6800 1400 50  0001 C CNN
+	1    6800 1400
+	0    1    1    0
+$EndComp
+Wire Wire Line
+	6800 1400 6750 1400
+Connection ~ 6800 1400
+Wire Wire Line
+	5950 1400 6150 1400
+Wire Wire Line
+	6150 1500 6150 1400
+Connection ~ 6150 1400
+$Comp
+L power:GND #PWR0160
+U 1 1 5F1C8E55
+P 6750 1500
+F 0 "#PWR0160" H 6750 1250 50  0001 C CNN
+F 1 "GND" H 6755 1327 50  0000 C CNN
+F 2 "" H 6750 1500 50  0001 C CNN
+F 3 "" H 6750 1500 50  0001 C CNN
+	1    6750 1500
+	1    0    0    -1
+$EndComp

Commit message: FPGA_ESP32 : esp32/rf pa+lna+switch routing progress
Parts:
- removed C20: 1uF, Capacitor_SMD:C_0402_1005Metric, symbol Device:C
- U3: value LP5910 -> LP5910-1.1BYKAT
Changed lines of the file:
@@
 P 6450 1300
 F 0 "U3" H 6450 1465 50  0000 C CNN
-F 1 "LP5910" H 6450 1374 50  0000 C CNN
+F 1 "LP5910-1.1BYKAT" H 6450 850 50  0000 C CNN
 F 2 "footprints:BGA-4_2x2_0.74x0.74mm" H 6450 1300 50  0001 C CNN
 F 3 "" H 6450 1300 50  0001 C CNN
@@
 $EndComp
 $Comp
-L Device:C C20
-U 1 1 5F192F78
-P 5950 1250
-F 0 "C20" H 6065 1296 50  0000 L CNN
-F 1 "1uF" H 6065 1205 50  0000 L CNN
-F 2 "Capacitor_SMD:C_0402_1005Metric" H 5988 1100 50  0001 C CNN
-F 3 "~" H 5950 1250 50  0001 C CNN
-	1    5950 1250
-	1    0    0    1
-$EndComp
-$Comp
-L power:GND #PWR0157
-U 1 1 5F192F7E
-P 5950 1100
-F 0 "#PWR0157" H 5950 850 50  0001 C CNN
-F 1 "GND" H 5955 927 50  0000 C CNN
-F 2 "" H 5950 1100 50  0001 C CNN
-F 3 "" H 5950 1100 50  0001 C CNN
-	1    5950 1100
-	1    0    0    1
-$EndComp
-$Comp
